File: Schematics/lower_lc_board/modules/power_module/power_module.kicad_sch (KiCad schematic)
At the start: 34 parts, among them J1 Stack Male Edge Connector, U1 TVS3300DRV, U10 ID_LM66100DCKR, U2 AMS1117, U3 ID_LM66100DCKR, U4 ID_LM66100DCKR

Commit message: more organizational work, add shared footprint, model, symbol dirs and clean up individuals
Parts:
- FB1: footprint BLM31KN121SN1L:BEADC3216X180N -> Resistor_SMD:R_0805_2012Metric
Other:
- title: Lower Board Power Module -> HYDRA | Power Circuitry
Changed lines of the file:
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@@
 	(paper "A4")
 	(title_block
-		(title "Lower Board Power Module")
-		(rev "B")
+		(title "HYDRA | Power Circuitry")
+		(rev "2")
 		(company "Queen's Rocket Engineering Team")
 		(comment 1 "Jeevan Sanchez")
@@
 			)
 		)
-		(property "Datasheet" "${KIPRJMOD}/../../Datasheets/ID-lm66100.pdf"
+		(property "Datasheet" "${KIPRJMOD}/../../Documentation/ideal_diode_lm66100_DS.pdf"
 			(at 170.18 40.64 0)
 			(effects
@@
 			)
 		)
-		(property "Datasheet" "${KIPRJMOD}/../../Datasheets/ID-lm66100.pdf"
+		(property "Datasheet" "${KIPRJMOD}/../../Documentation/ideal_diode_lm66100_DS.pdf"
 			(at 170.18 83.82 0)
 			(effects
@@
 			)
 		)
-		(property "Datasheet" "${KIPRJMOD}/../../Datasheets/ID-lm66100.pdf"
+		(property "Datasheet" "${KIPRJMOD}/../../Documentation/ideal_diode_lm66100_DS.pdf"
 			(at 170.18 63.5 0)
 			(effects
@@
 			)
 		)
-		(property "Datasheet" "${KIPRJMOD}/../../Datasheets/SURGE-PROT-tvs3300.pdf"
+		(property "Datasheet" "${KIPRJMOD}/../../Documentation/surgeprot_tvs3300_DS.pdf"
 			(at 54.61 142.24 0)
 			(effects
@@
 			)
 		)
-		(property "Footprint" "BLM31KN121SN1L:BEADC3216X180N"
+		(property "Footprint" "Resistor_SMD:R_0805_2012Metric"
 			(at 72.39 136.398 90)
 			(effects
@@
 			)
 		)
-		(property "Datasheet" "${KIPRJMOD}/../../Datasheets/FERRITEB-A700000010386127.pdf"
+		(property "Datasheet" ""
 			(at 72.39 134.62 0)
 			(effects
@@
 			)
 		)
-		(property "Datasheet" "http://www.advanced-monolithic.com/pdf/ds1117.pdf"
+		(property "Datasheet" "${KIPRJMOD}/../../Documentation/LDO_ds1117_DS.pdf"
 			(at 162.56 140.97 0)
 			(effects
