File: Schematics/shared_schematics/VALVE_control.kicad_sch (KiCad schematic)
At the start: 7 parts, among them J2 SOL_CONN, Q1 AO3400A

Commit message: review of schematics and pcb
- verified all STM pins
- reviewed all circuits
- reviewed trace clearences, made sure routes are connected, etc.
Parts:
- C16: JLCPCB (none) -> C13585
- J2: Digikey 900-0530470260-ND -> 455-B02B-PASK-1-ND
- Q1: JLCPCB (none) -> C20917
Changed lines of the file:
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@@
+			)
+		)
+		(property "JLCPCB" "C20917"
+			(at 201.93 93.98 0)
+			(effects
+				(font
+					(size 1.27 1.27)
+				)
+				(hide yes)
 			)
 		)
@@
 			)
 		)
+		(property "JLCPCB" "C13585"
+			(at 137.16 93.98 0)
+			(effects
+				(font
+					(size 1.27 1.27)
+				)
+				(hide yes)
+			)
+		)
 		(pin "2"
 		)
@@
 			)
 		)
-		(property "Digikey" "900-0530470260-ND"
+		(property "Digikey" "455-B02B-PASK-1-ND"
 			(at 151.13 93.98 90)
 			(effects

Commit message: increase width on power rails from USB and SWD, start tuning diff pairs
Parts:
- R36: JLCPCB (none) -> C8218
Changed lines of the file:
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@@
+			)
+		)
+		(property "JLCPCB" "C8218"
+			(at 184.15 93.98 0)
+			(effects
+				(font
+					(size 1.27 1.27)
+				)
+				(hide yes)
 			)
 		)

Commit message: refactor with new conns
Parts:
- J7: renamed from J2; footprint ul_B02B-PASK-1:CONN_B02B-PASK-1_JST -> NANO-V-2-CONN:MOLEX_1053091102
- renumbered C16 to C20, C15 to C21, D16 to D14, Q1 to Q2, R36 to R26, R39 to R31
Changed lines of the file:
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@@
 		(shape input)
 		(at 204.47 81.28 90)
+		(fields_autoplaced yes)
 		(effects
 			(font
@@
 		(shape input)
 		(at 201.93 88.9 180)
+		(fields_autoplaced yes)
 		(effects
 			(font
@@
 		(shape input)
 		(at 180.34 93.98 180)
+		(fields_autoplaced yes)
 		(effects
 			(font
@@
 		(shape input)
 		(at 151.13 99.06 270)
+		(fields_autoplaced yes)
 		(effects
 			(font
@@
 		(shape input)
 		(at 139.7 99.06 270)
+		(fields_autoplaced yes)
 		(effects
 			(font
@@
 		(shape input)
 		(at 153.67 99.06 270)
+		(fields_autoplaced yes)
 		(effects
 			(font
@@
 		(shape input)
 		(at 207.01 88.9 0)
+		(fields_autoplaced yes)
 		(effects
 			(font
@@
 		(shape input)
 		(at 180.34 93.98 180)
+		(fields_autoplaced yes)
 		(effects
 			(font
@@
 		(dnp no)
 		(fields_autoplaced yes)
-		(property "Reference" "Q1"
+		(property "Reference" "Q2"
 			(at 208.28 92.7099 0)
 			(effects
@@
 		)
 		(instances
+			(project ""
+				(path "/8de962ac-ee95-4233-a205-efbcd04063bc/bb8d84b9-ecb3-4da4-948c-d0cf2dc1ed2d/94e68ee1-e1f2-4047-b299-1f0f2281affb"
+					(reference "Q1")
+					(unit 1)
+				)
+				(path "/8de962ac-ee95-4233-a205-efbcd04063bc/bb8d84b9-ecb3-4da4-948c-d0cf2dc1ed2d/cf6cc7ca-f6f8-4955-86eb-3247d55d8f2c"
+					(reference "Q2")
+					(unit 1)
+				)
+			)
 			(project "upper_lc_board"
 				(path "/9b1a1d2a-fad7-4f10-83f3-1f83e9656c75/f003a3ad-0ca0-4253-bb6a-1aee93b0e37f/1bd8ce37-8ddd-4ff8-9ae8-5224bdd9bb9e"
@@
 		(dnp no)
 		(fields_autoplaced yes)
-		(property "Reference" "D16"
+		(property "Reference" "D14"
 			(at 207.01 83.5024 90)
 			(effects
@@
 		)
 		(instances
+			(project ""
+				(path "/8de962ac-ee95-4233-a205-efbcd04063bc/bb8d84b9-ecb3-4da4-948c-d0cf2dc1ed2d/94e68ee1-e1f2-4047-b299-1f0f2281affb"
+					(reference "D13")
+					(unit 1)
+				)
+				(path "/8de962ac-ee95-4233-a205-efbcd04063bc/bb8d84b9-ecb3-4da4-948c-d0cf2dc1ed2d/cf6cc7ca-f6f8-4955-86eb-3247d55d8f2c"
+					(reference "D14")
+					(unit 1)
+				)
+			)
 			(project "upper_lc_board"
 				(path "/9b1a1d2a-fad7-4f10-83f3-1f83e9656c75/f003a3ad-0ca0-4253-bb6a-1aee93b0e37f/1bd8ce37-8ddd-4ff8-9ae8-5224bdd9bb9e"
@@
 		(instances
 			(project ""
+				(path "/8de962ac-ee95-4233-a205-efbcd04063bc/bb8d84b9-ecb3-4da4-948c-d0cf2dc1ed2d/94e68ee1-e1f2-4047-b299-1f0f2281affb"
+					(reference "#PWR0123")
+					(unit 1)
+				)
+				(path "/8de962ac-ee95-4233-a205-efbcd04063bc/bb8d84b9-ecb3-4da4-948c-d0cf2dc1ed2d/cf6cc7ca-f6f8-4955-86eb-3247d55d8f2c"
+					(reference "#PWR051")
+					(unit 1)
+				)
+			)
+			(project ""
 				(path "/9b1a1d2a-fad7-4f10-83f3-1f83e9656c75/f003a3ad-0ca0-4253-bb6a-1aee93b0e37f/1bd8ce37-8ddd-4ff8-9ae8-5224bdd9bb9e"
 					(reference "#PWR0123")
@@
 		(on_board yes)
 		(dnp no)
-		(property "Reference" "C16"
+		(property "Reference" "C20"
 			(at 132.08 90.17 0)
 			(effects
@@
 		)
 		(instances
+			(project ""
+				(path "/8de962ac-ee95-4233-a205-efbcd04063bc/bb8d84b9-ecb3-4da4-948c-d0cf2dc1ed2d/94e68ee1-e1f2-4047-b299-1f0f2281affb"
+					(reference "C18")
+					(unit 1)
+				)
+				(path "/8de962ac-ee95-4233-a205-efbcd04063bc/bb8d84b9-ecb3-4da4-948c-d0cf2dc1ed2d/cf6cc7ca-f6f8-4955-86eb-3247d55d8f2c"
+					(reference "C20")
+					(unit 1)
+				)
+			)
 			(project ""
 				(path "/9b1a1d2a-fad7-4f10-83f3-1f83e9656c75/f003a3ad-0ca0-4253-bb6a-1aee93b0e37f/1bd8ce37-8ddd-4ff8-9ae8-5224bdd9bb9e"
@@
 		(on_board yes)
 		(dnp no)
-		(property "Reference" "R39"
+		(property "Reference" "R31"
 			(at 189.23 97.79 0)
 			(effects
@@
 		)
 		(instances
+			(project ""
+				(path "/8de962ac-ee95-4233-a205-efbcd04063bc/bb8d84b9-ecb3-4da4-948c-d0cf2dc1ed2d/94e68ee1-e1f2-4047-b299-1f0f2281affb"
+					(reference "R20")
+					(unit 1)
+				)
+				(path "/8de962ac-ee95-4233-a205-efbcd04063bc/bb8d84b9-ecb3-4da4-948c-d0cf2dc1ed2d/cf6cc7ca-f6f8-4955-86eb-3247d55d8f2c"
+					(reference "R31")
+					(unit 1)
+				)
+			)
 			(project "upper_lc_board"
 				(path "/9b1a1d2a-fad7-4f10-83f3-1f83e9656c75/f003a3ad-0ca0-4253-bb6a-1aee93b0e37f/1bd8ce37-8ddd-4ff8-9ae8-5224bdd9bb9e"
@@
 		(on_board yes)
 		(dnp no)
-		(property "Reference" "R36"
+		(property "Reference" "R26"
 			(at 184.15 96.52 90)
 			(effects
@@
 		)
 		(instances
+			(project ""
+				(path "/8de962ac-ee95-4233-a205-efbcd04063bc/bb8d84b9-ecb3-4da4-948c-d0cf2dc1ed2d/94e68ee1-e1f2-4047-b299-1f0f2281affb"
+					(reference "R19")
+					(unit 1)
+				)
+				(path "/8de962ac-ee95-4233-a205-efbcd04063bc/bb8d84b9-ecb3-4da4-948c-d0cf2dc1ed2d/cf6cc7ca-f6f8-4955-86eb-3247d55d8f2c"
+					(reference "R26")
+					(unit 1)
+				)
+			)
 			(project "upper_lc_board"
 				(path "/9b1a1d2a-fad7-4f10-83f3-1f83e9656c75/f003a3ad-0ca0-4253-bb6a-1aee93b0e37f/1bd8ce37-8ddd-4ff8-9ae8-5224bdd9bb9e"
@@
 		)
 		(instances
+			(project ""
+				(path "/8de962ac-ee95-4233-a205-efbcd04063bc/bb8d84b9-ecb3-4da4-948c-d0cf2dc1ed2d/94e68ee1-e1f2-4047-b299-1f0f2281affb"
+					(reference "#PWR0125")
+					(unit 1)
+				)
+				(path "/8de962ac-ee95-4233-a205-efbcd04063bc/bb8d84b9-ecb3-4da4-948c-d0cf2dc1ed2d/cf6cc7ca-f6f8-4955-86eb-3247d55d8f2c"
+					(reference "#PWR080")
+					(unit 1)
+				)
+			)
 			(project "upper_lc_board"
 				(path "/9b1a1d2a-fad7-4f10-83f3-1f83e9656c75/f003a3ad-0ca0-4253-bb6a-1aee93b0e37f/1bd8ce37-8ddd-4ff8-9ae8-5224bdd9bb9e"
@@
 		(on_board yes)
 		(dnp no)
-		(property "Reference" "J2"
+		(property "Reference" "J7"
 			(at 156.21 92.7099 90)
 			(effects
@@
 			)
 		)
-		(property "Footprint" "ul_B02B-PASK-1:CONN_B02B-PASK-1_JST"
+		(property "Footprint" "NANO-V-2-CONN:MOLEX_1053091102"
 			(at 151.13 93.98 0)
 			(effects
@@
 		)
 		(instances
+			(project ""
+				(path "/8de962ac-ee95-4233-a205-efbcd04063bc/bb8d84b9-ecb3-4da4-948c-d0cf2dc1ed2d/94e68ee1-e1f2-4047-b299-1f0f2281affb"
+					(reference "J7")
+					(unit 1)
+				)
+				(path "/8de962ac-ee95-4233-a205-efbcd04063bc/bb8d84b9-ecb3-4da4-948c-d0cf2dc1ed2d/cf6cc7ca-f6f8-4955-86eb-3247d55d8f2c"
+					(reference "J6")
+					(unit 1)
+				)
+			)
 			(project ""
 				(path "/9b1a1d2a-fad7-4f10-83f3-1f83e9656c75/f003a3ad-0ca0-4253-bb6a-1aee93b0e37f/1bd8ce37-8ddd-4ff8-9ae8-5224bdd9bb9e"
@@
 		(on_board yes)
 		(dnp no)
-		(property "Reference" "C15"
+		(property "Reference" "C21"
 			(at 132.334 94.996 0)
 			(effects
@@
 		)
 		(instances
+			(project ""
+				(path "/8de962ac-ee95-4233-a205-efbcd04063bc/bb8d84b9-ecb3-4da4-948c-d0cf2dc1ed2d/94e68ee1-e1f2-4047-b299-1f0f2281affb"
+					(reference "C19")
+					(unit 1)
+				)
+				(path "/8de962ac-ee95-4233-a205-efbcd04063bc/bb8d84b9-ecb3-4da4-948c-d0cf2dc1ed2d/cf6cc7ca-f6f8-4955-86eb-3247d55d8f2c"
+					(reference "C21")
+					(unit 1)
+				)
+			)
 			(project ""
 				(path "/9b1a1d2a-fad7-4f10-83f3-1f83e9656c75/f003a3ad-0ca0-4253-bb6a-1aee93b0e37f/1bd8ce37-8ddd-4ff8-9ae8-5224bdd9bb9e"
@@
 		)
 		(instances
+			(project ""
+				(path "/8de962ac-ee95-4233-a205-efbcd04063bc/bb8d84b9-ecb3-4da4-948c-d0cf2dc1ed2d/94e68ee1-e1f2-4047-b299-1f0f2281affb"
+					(reference "#PWR0124")
+					(unit 1)
+				)
+				(path "/8de962ac-ee95-4233-a205-efbcd04063bc/bb8d84b9-ecb3-4da4-948c-d0cf2dc1ed2d/cf6cc7ca-f6f8-4955-86eb-3247d55d8f2c"
+					(reference "#PWR052")
+					(unit 1)
+				)
+			)
 			(project "upper_lc_board"
 				(path "/9b1a1d2a-fad7-4f10-83f3-1f83e9656c75/f003a3ad-0ca0-4253-bb6a-1aee93b0e37f/1bd8ce37-8ddd-4ff8-9ae8-5224bdd9bb9e"

Commit message: layout updates after review, cleaned up schematic organization
Parts:
- renumbered C20 to C18, C21 to C19, D14 to D13, Q2 to Q1, R26 to R19, R31 to R20
Changed lines of the file:
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@@
 		(dnp no)
 		(fields_autoplaced yes)
-		(property "Reference" "Q2"
+		(property "Reference" "Q1"
 			(at 208.28 92.7099 0)
 			(effects
@@
 		)
 		(instances
-			(project ""
+			(project "upper_lc_board_v2"
 				(path "/8de962ac-ee95-4233-a205-efbcd04063bc/bb8d84b9-ecb3-4da4-948c-d0cf2dc1ed2d/94e68ee1-e1f2-4047-b299-1f0f2281affb"
 					(reference "Q1")
@@
 		(dnp no)
 		(fields_autoplaced yes)
-		(property "Reference" "D14"
+		(property "Reference" "D13"
 			(at 207.01 83.5024 90)
 			(effects
@@
 		)
 		(instances
-			(project ""
+			(project "upper_lc_board_v2"
 				(path "/8de962ac-ee95-4233-a205-efbcd04063bc/bb8d84b9-ecb3-4da4-948c-d0cf2dc1ed2d/94e68ee1-e1f2-4047-b299-1f0f2281affb"
 					(reference "D13")
@@
 		)
 		(instances
-			(project ""
+			(project "upper_lc_board_v2"
 				(path "/8de962ac-ee95-4233-a205-efbcd04063bc/bb8d84b9-ecb3-4da4-948c-d0cf2dc1ed2d/94e68ee1-e1f2-4047-b299-1f0f2281affb"
 					(reference "#PWR0123")
@@
 		(on_board yes)
 		(dnp no)
-		(property "Reference" "C20"
+		(property "Reference" "C18"
 			(at 132.08 90.17 0)
 			(effects
@@
 		)
 		(instances
-			(project ""
+			(project "upper_lc_board_v2"
 				(path "/8de962ac-ee95-4233-a205-efbcd04063bc/bb8d84b9-ecb3-4da4-948c-d0cf2dc1ed2d/94e68ee1-e1f2-4047-b299-1f0f2281affb"
 					(reference "C18")
@@
 		(on_board yes)
 		(dnp no)
-		(property "Reference" "R31"
+		(property "Reference" "R20"
 			(at 189.23 97.79 0)
 			(effects
@@
 		)
 		(instances
-			(project ""
+			(project "upper_lc_board_v2"
 				(path "/8de962ac-ee95-4233-a205-efbcd04063bc/bb8d84b9-ecb3-4da4-948c-d0cf2dc1ed2d/94e68ee1-e1f2-4047-b299-1f0f2281affb"
 					(reference "R20")
@@
 		(on_board yes)
 		(dnp no)
-		(property "Reference" "R26"
+		(property "Reference" "R19"
 			(at 184.15 96.52 90)
 			(effects
@@
 		)
 		(instances
-			(project ""
+			(project "upper_lc_board_v2"
 				(path "/8de962ac-ee95-4233-a205-efbcd04063bc/bb8d84b9-ecb3-4da4-948c-d0cf2dc1ed2d/94e68ee1-e1f2-4047-b299-1f0f2281affb"
 					(reference "R19")
@@
 		)
 		(instances
-			(project ""
+			(project "upper_lc_board_v2"
 				(path "/8de962ac-ee95-4233-a205-efbcd04063bc/bb8d84b9-ecb3-4da4-948c-d0cf2dc1ed2d/94e68ee1-e1f2-4047-b299-1f0f2281affb"
 					(reference "#PWR0125")
@@
 		)
 		(instances
-			(project ""
+			(project "upper_lc_board_v2"
 				(path "/8de962ac-ee95-4233-a205-efbcd04063bc/bb8d84b9-ecb3-4da4-948c-d0cf2dc1ed2d/94e68ee1-e1f2-4047-b299-1f0f2281affb"
 					(reference "J7")
@@
 		(on_board yes)
 		(dnp no)
-		(property "Reference" "C21"
+		(property "Reference" "C19"
 			(at 132.334 94.996 0)
 			(effects
@@
 		)
 		(instances
-			(project ""
+			(project "upper_lc_board_v2"
 				(path "/8de962ac-ee95-4233-a205-efbcd04063bc/bb8d84b9-ecb3-4da4-948c-d0cf2dc1ed2d/94e68ee1-e1f2-4047-b299-1f0f2281affb"
 					(reference "C19")
@@
 		)
 		(instances
-			(project ""
+			(project "upper_lc_board_v2"
 				(path "/8de962ac-ee95-4233-a205-efbcd04063bc/bb8d84b9-ecb3-4da4-948c-d0cf2dc1ed2d/94e68ee1-e1f2-4047-b299-1f0f2281affb"
 					(reference "#PWR0124")

Commit message: swap I2C lines, add digi numbers to conns, fix diode issue
Parts:
- J7: Digikey 455-B02B-PASK-1-ND -> WM14965-ND
Changed lines of the file:
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@@
 			)
 		)
-		(property "Digikey" "455-B02B-PASK-1-ND"
+		(property "Digikey" "WM14965-ND"
 			(at 151.13 93.98 90)
 			(effects

Commit message: updated part numbers and fixed minor circuit issues
Parts:
- C18: JLCPCB C13585 -> (none); LCSC (none) -> C13585
- C19: JLCPCB C14663 -> (none); LCSC (none) -> C14663
- Q1: JLCPCB C20917 -> (none)
- R19: JLCPCB C8218 -> (none)
Changed lines of the file:
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@@
-			)
-		)
-		(property "JLCPCB" "C20917"
-			(at 201.93 93.98 0)
-			(effects
-				(font
-					(size 1.27 1.27)
-				)
-				(hide yes)
 			)
 		)
@@
 			)
 		)
-		(property "JLCPCB" "C13585"
+		(property "LCSC" "C13585"
 			(at 137.16 93.98 0)
 			(effects
@@
 					(size 1.27 1.27)
 				)
-				(hide yes)
 			)
 		)
@@
 			)
 		)
-		(property "JLCPCB" "C8218"
-			(at 184.15 93.98 0)
-			(effects
-				(font
-					(size 1.27 1.27)
-				)
-				(hide yes)
-			)
-		)
 		(pin "2"
 		)
@@
 			)
 		)
-		(property "JLCPCB" "C14663"
+		(property "LCSC" "C14663"
 			(at 142.24 93.98 0)
 			(effects
