File: Schematics/shared_schematics/TC_module.kicad_sch (KiCad schematic)
At the start: 11 parts, among them J7 Screw_Terminal_01x02

Commit message: ADC routing
Parts:
- R29, R40: footprint Resistor_SMD:R_0603_1608Metric -> Resistor_SMD:R_0402_1005Metric
Changed lines of the file:
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@@
 			)
 		)
-		(property "Footprint" "Resistor_SMD:R_0603_1608Metric"
+		(property "Footprint" "Resistor_SMD:R_0402_1005Metric"
 			(at 154.432 104.14 90)
 			(effects
@@
 			)
 		)
-		(property "Footprint" "Resistor_SMD:R_0603_1608Metric"
+		(property "Footprint" "Resistor_SMD:R_0402_1005Metric"
 			(at 146.812 104.14 90)
 			(effects

Commit message: routing work
Parts:
- R24: footprint Resistor_SMD:R_1206_3216Metric_Pad1.30x1.75mm_HandSolder -> Resistor_SMD:R_0805_2012Metric
Changed lines of the file:
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@@
 			)
 		)
-		(property "Footprint" "Resistor_SMD:R_1206_3216Metric_Pad1.30x1.75mm_HandSolder"
+		(property "Footprint" "Resistor_SMD:R_0805_2012Metric"
 			(at 150.368 86.36 90)
 			(effects

Commit message: testing work
Parts:
- R24: footprint Resistor_SMD:R_0805_2012Metric -> Resistor_SMD:R_0603_1608Metric
- R28: footprint Resistor_SMD:R_1206_3216Metric_Pad1.30x1.75mm_HandSolder -> Resistor_SMD:R_0603_1608Metric
Changed lines of the file:
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@@
 			)
 		)
-		(property "Footprint" "Resistor_SMD:R_0805_2012Metric"
+		(property "Footprint" "Resistor_SMD:R_0603_1608Metric"
 			(at 150.368 86.36 90)
 			(effects
@@
 			)
 		)
-		(property "Footprint" "Resistor_SMD:R_1206_3216Metric_Pad1.30x1.75mm_HandSolder"
+		(property "Footprint" "Resistor_SMD:R_0603_1608Metric"
 			(at 157.988 86.36 90)
 			(effects

Commit message: remove AGND
simplicity
Connections:
- net GNDA renamed GND

Commit message: ADC testing
- update testing FW with new ADC lib
- switched 165 shunt resistor to 60 based on fixed calculations
Parts:
- renumbered C30 to C28, C31 to C29, C32 to C30, D18 to D19, R26 to R19, R24 to R20, R29 to R24, R28 to R25, R40 to R26
Connections:
- net +3V3: now also D19.2 (K2); no longer D19.5 (K4)
- net GND: now also D19.1 (A1); no longer D19.4 (A3)
- net at R25.1, R26.1: now also D19.6 (K3A4); no longer D19.3 (K1A2)

Commit message: adjust routing for 0603 min. footprints
Parts:
- R24, R26: footprint Resistor_SMD:R_0402_1005Metric -> Resistor_SMD:R_0603_1608Metric
Changed lines of the file:
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@@
 			)
 		)
-		(property "Footprint" "Resistor_SMD:R_0402_1005Metric"
+		(property "Footprint" "Resistor_SMD:R_0603_1608Metric"
 			(at 154.432 104.14 90)
 			(effects
@@
 			)
 		)
-		(property "Footprint" "Resistor_SMD:R_0402_1005Metric"
+		(property "Footprint" "Resistor_SMD:R_0603_1608Metric"
 			(at 146.812 104.14 90)
 			(effects

Commit message: review of schematics and pcb
- verified all STM pins
- reviewed all circuits
- reviewed trace clearences, made sure routes are connected, etc.
Parts:
- C29, C30: JLCPCB (none) -> C1588
- R20, R25: JLCPCB (none) -> C21190; LCSC C4410 -> C21190
Changed lines of the file:
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@@
 			)
 		)
-		(property "LCSC" "C4410"
+		(property "LCSC" "C21190"
 			(at 148.59 86.36 90)
+			(effects
+				(font
+					(size 1.27 1.27)
+				)
+				(hide yes)
+			)
+		)
+		(property "JLCPCB" "C21190"
+			(at 148.59 86.36 0)
 			(effects
 				(font
@@
 		)
 		(property "Description" "Unpolarized capacitor"
+			(at 194.31 97.79 0)
+			(effects
+				(font
+					(size 1.27 1.27)
+				)
+				(hide yes)
+			)
+		)
+		(property "JLCPCB" "C1588"
 			(at 194.31 97.79 0)
 			(effects
@@
 			)
 		)
+		(property "JLCPCB" "C1588"
+			(at 194.31 87.63 0)
+			(effects
+				(font
+					(size 1.27 1.27)
+				)
+				(hide yes)
+			)
+		)
 		(pin "2"
 		)
@@
 			)
 		)
-		(property "LCSC" "C4410"
+		(property "LCSC" "C21190"
 			(at 156.21 86.36 90)
 			(effects
 				(font
+					(size 1.27 1.27)
+				)
+				(hide yes)
+			)
+		)
+		(property "JLCPCB" "C21190"
+			(at 156.21 86.36 0)
+			(effects
+				(font

Commit message: increase width on power rails from USB and SWD, start tuning diff pairs
Parts:
- D18, D19: JLCPCB (none) -> BAV199DW
- R19, R27: JLCPCB (none) -> C22935
- R24, R26: JLCPCB (none) -> C8218
Changed lines of the file:
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@@
+			)
+		)
+		(property "JLCPCB" "C22935"
+			(at 139.7 81.28 0)
+			(effects
+				(font
+					(size 1.27 1.27)
+				)
+				(hide yes)
 			)
 		)
@@
 		)
 		(property "LCSC" "C22935"
+			(at 166.37 81.28 0)
+			(effects
+				(font
+					(size 1.27 1.27)
+				)
+				(hide yes)
+			)
+		)
+		(property "JLCPCB" "C22935"
 			(at 166.37 81.28 0)
 			(effects
@@
 			)
 		)
+		(property "JLCPCB" "C8218"
+			(at 156.21 104.14 0)
+			(effects
+				(font
+					(size 1.27 1.27)
+				)
+				(hide yes)
+			)
+		)
 		(pin "1"
 		)
@@
 			)
 		)
+		(property "JLCPCB" "BAV199DW"
+			(at 163.83 97.79 0)
+			(effects
+				(font
+					(size 1.27 1.27)
+				)
+				(hide yes)
+			)
+		)
 		(pin "6"
 		)
@@
 		)
 		(property "LCSC" "C459846"
+			(at 139.7 97.79 0)
+			(effects
+				(font
+					(size 1.27 1.27)
+				)
+				(hide yes)
+			)
+		)
+		(property "JLCPCB" "BAV199DW"
 			(at 139.7 97.79 0)
 			(effects
@@
 			(at 148.59 104.14 0)
 			(effects
+				(font
+					(size 1.27 1.27)
+				)
+				(hide yes)
+			)
+		)
+		(property "JLCPCB" "C8218"
+			(at 148.59 104.14 0)
+			(effects
