File: Schematics/upper_lc_board/upper_lc_board.kicad_pcb (KiCad board)
At the start: 4 copper layers, 69.5 x 60 mm, 107 parts, among them J1 Stack Male Edge Connector, J2 SOL1_CONN, J3 PT1, J4 PT1, J5 HALL, J6 SOL2_CONN, J7 Screw_Terminal_01x02, J8 USB_C_Female_USB2_Small, Q1 AO3400A, Q2 AO3400A, SW1 SW_ESP_BOOT_MODE, SW2 SW_ESP_RESET, U1 ESP32-S3-WROOM-1-N16, U2 ISO1044BDR, U3 AMS1117-3.3, U4 ID_LM66100DCKR, U5 ID_LM66100DCKR, U7 ADC_ADS131M04IPWR, U9 TVS3300DRV

Commit message: fix CAN transceiver model
Other:
- board text added: "PHOENIX"
- board text removed: "PHEONIX"
Changed lines of the file:
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@@
 			(pintype "power_in")
 		)
-		(model "${KIPRJMOD}/models/ISO1042BDWVR.step"
+		(model "${KIPRJMOD}/models/D0008A.stp"
 			(offset
 				(xyz 0 0 0)
@@
 			)
 			(rotate
-				(xyz -90 0 0)
+				(xyz 0 0 0)
 			)
 		)
@@
 		)
 	)
-	(gr_text "PHEONIX"
+	(gr_text "PHOENIX"
 		(at 98.73 122.31 90)
 		(layer "F.SilkS" knockout)
