File: Schematics/upper_lc_board/upper_lc_board.kicad_pcb (KiCad board)
At the start: 4 copper layers, 69.5 x 60 mm, 108 parts, among them J1 USB_C_Female_USB2_Small, J2 Stack Male Edge Connector, J3 PT, J4 PT, J5 HALL-1, J6 SOL_CONN, J7 SOL_CONN, Q1 AO3400A, Q2 AO3400A, Q4 2N7002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

Commit message: added 24V sensing to upper board
Parts:
- removed C27: 0.1uF, Capacitor_SMD:C_0603_1608Metric
- added R27: 33, Resistor_SMD:R_0603_1608Metric, F.Cu at (136.1, 98.1)
- added R30: 100k, Resistor_SMD:R_0603_1608Metric, F.Cu at (154.3, 105.0)
- added R32: 10k, Resistor_SMD:R_0603_1608Metric, F.Cu at (154.4, 103.3)
- R8: footprint Resistor_SMD:R_1206_3216Metric_Pad1.30x1.75mm_HandSolder -> Resistor_SMD:R_0603_1608Metric
Connections:
- net /ESP32-S3 Breakout Circuitry/GPIO_01 renamed /ESP32-S3 Breakout Circuitry/CAN_TX
- net /ESP32-S3 Breakout Circuitry/GPIO_02 renamed /ESP32-S3 Breakout Circuitry/CAN_RX
- net /ESP32-S3 Breakout Circuitry/GPIO_35 renamed /ESP32-S3 Breakout Circuitry/WIFI_LED
- net /ESP32-S3 Breakout Circuitry/GPIO_36 renamed /ESP32-S3 Breakout Circuitry/CAN_LED
- net /ESP32-S3 Breakout Circuitry/GPIO_37 renamed /ESP32-S3 Breakout Circuitry/DEBUG_LED
- net /ESP32-S3 Breakout Circuitry/GPIO_42 renamed /ESP32-S3 Breakout Circuitry/RGB_DATAIN
- net BUZZ_IN renamed /ESP32-S3 Breakout Circuitry/BUZZ_IN
- U1 pad 15: /ESP32-S3 Breakout Circuitry/GPIO_03 -> unconnected-(U1-IO3-Pad15)
- U1 pad 16: /ESP32-S3 Breakout Circuitry/GPIO_46 -> unconnected-(U1-IO46-Pad16)
- U1 pad 19: ADC_CLKIN -> Net-(U1-IO11)
- U1 pad 26: /ESP32-S3 Breakout Circuitry/GPIO_45 -> unconnected-(U1-IO45-Pad26)
- U1 pad 31: /ESP32-S3 Breakout Circuitry/GPIO_38 -> unconnected-(U1-IO38-Pad31)
- U1 pad 32: /ESP32-S3 Breakout Circuitry/GPIO_39 -> unconnected-(U1-IO39-Pad32)
- U1 pad 33: /ESP32-S3 Breakout Circuitry/GPIO_40 -> unconnected-(U1-IO40-Pad33)
- U1 pad 7: unconnected-(U1-IO7-Pad7) -> 24V_SENSE
Routing:
- net 24V_SENSE: track 0.00 -> 16.3 mm, vias 0 -> 2
- net +24V: track 137.9 -> 150.0 mm, vias 4 -> 5
- net GND: track 132.5 -> 129.0 mm, vias 256 -> 257
- net ADC_CLKIN: track 11.8 -> 8.75 mm
- net Net-(U1-IO11): track 0.00 -> 2.13 mm

Commit message: add ed pinouts
Connections:
- net SPI_MISO renamed ADC_MISO
- net SPI_MOSI renamed ADC_MOSI
- net SPI_SCLK renamed ADC_SCLK
- net VALVE1_CTRL renamed SOL1_EN
- net VALVE2_CTRL renamed SOL2_EN
- net VPT-SW renamed VPT_EN
Changed lines of the file:
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@@
 	(net 40 "unconnected-(J2-BATT_B-PadB7)")
 	(net 41 "unconnected-(J2-Reserved-PadB18)")
-	(net 42 "unconnected-(J2-BATT_B-PadB7)_2")
+	(net 42 "unconnected-(J2-BATT_A-PadB1)_0")
 	(net 43 "unconnected-(J2-BATT_A-PadB1)_1")
 	(net 44 "unconnected-(J2-BATT_B-PadB7)_1")
@@
 	(net 46 "HALL_SCL")
 	(net 47 "HALL_SDA")
-	(net 48 "unconnected-(J2-3.3V_B-PadA7)_1")
-	(net 49 "unconnected-(J2-BATT_A-PadB1)_2")
+	(net 48 "unconnected-(J2-GND_B-PadA12)_0")
+	(net 49 "unconnected-(J2-BATT_B-PadB7)_0")
 	(net 50 "Net-(Q2-G)")
 	(net 51 "/ESP32-S3 Breakout Circuitry/RGB_DATAIN")
@@
 	(net 53 "Net-(J1-CC2)")
 	(net 54 "+24V")
-	(net 55 "VALVE1_CTRL")
-	(net 56 "VALVE2_CTRL")
-	(net 57 "VPT-SW")
+	(net 55 "unconnected-(J2-3.3V_B-PadA7)_0")
+	(net 56 "SOL1_EN")
+	(net 57 "SOL2_EN")
 	(net 58 "unconnected-(U1-TXD0-Pad37)")
 	(net 59 "unconnected-(U1-RXD0-Pad36)")
@@
 	(net 67 "Net-(BZ1--)")
 	(net 68 "Net-(Q4-G)")
-	(net 69 "SPI_SCLK")
-	(net 70 "SPI_MISO")
-	(net 71 "SPI_MOSI")
+	(net 69 "VPT_EN")
+	(net 70 "ADC_SCLK")
+	(net 71 "ADC_MISO")
 	(net 72 "ADC_CLKIN")
 	(net 73 "ADC_DRDY")
@@
 	(net 79 "unconnected-(J1-SBU1-PadA8)")
 	(net 80 "unconnected-(J1-SBU2-PadB8)")
-	(net 81 "unconnected-(J2-GND_B-PadA12)_4")
+	(net 81 "ADC_MOSI")
 	(net 82 "Net-(J3-Pin_2)")
 	(net 83 "Net-(Q1-G)")
@@
 			(layers "F.Cu" "F.Paste" "F.Mask")
 			(roundrect_rratio 0.125)
-			(net 69 "SPI_SCLK")
+			(net 70 "ADC_SCLK")
 			(pinfunction "SCLK")
 			(pintype "input")
@@
 			(layers "F.Cu" "F.Paste" "F.Mask")
 			(roundrect_rratio 0.125)
-			(net 70 "SPI_MISO")
+			(net 71 "ADC_MISO")
 			(pinfunction "DOUT")
 			(pintype "output")
@@
 			(layers "F.Cu" "F.Paste" "F.Mask")
 			(roundrect_rratio 0.125)
-			(net 71 "SPI_MOSI")
+			(net 81 "ADC_MOSI")
 			(pinfunction "DIN")
 			(pintype "input")
@@
 			(size 0.7 4.3)
 			(layers "B.Cu" "B.Mask")
-			(net 48 "unconnected-(J2-3.3V_B-PadA7)_1")
+			(net 55 "unconnected-(J2-3.3V_B-PadA7)_0")
 			(pinfunction "3.3V_B")
 			(pintype "passive+no_connect")
@@
 			(size 0.7 4.3)
 			(layers "B.Cu" "B.Mask")
-			(net 86 "unconnected-(J2-GND_B-PadA12)_2")
+			(net 85 "unconnected-(J2-GND_B-PadA12)_1")
 			(pinfunction "GND_B")
 			(pintype "passive+no_connect")
@@
 			(size 0.7 4.3)
 			(layers "B.Cu" "B.Mask")
-			(net 87 "unconnected-(J2-GND_B-PadA12)_3")
+			(net 86 "unconnected-(J2-GND_B-PadA12)_2")
 			(pinfunction "GND_B")
 			(pintype "power_in+no_connect")
@@
 			(size 0.7 4.3)
 			(layers "F.Cu" "F.Mask")
-			(net 49 "unconnected-(J2-BATT_A-PadB1)_2")
+			(net 43 "unconnected-(J2-BATT_A-PadB1)_1")
 			(pinfunction "BATT_A")
 			(pintype "power_out+no_connect")
@@
 			(size 0.7 4.3)
 			(layers "F.Cu" "F.Mask")
-			(net 43 "unconnected-(J2-BATT_A-PadB1)_1")
+			(net 42 "unconnected-(J2-BATT_A-PadB1)_0")
 			(pinfunction "BATT_A")
 			(pintype "passive+no_connect")
@@
 			(size 0.7 4.3)
 			(layers "F.Cu" "F.Mask")
-			(net 44 "unconnected-(J2-BATT_B-PadB7)_1")
+			(net 49 "unconnected-(J2-BATT_B-PadB7)_0")
 			(pinfunction "BATT_B")
 			(pintype "power_out+no_connect")
@@
 			(size 0.7 4.3)
 			(layers "F.Cu" "F.Mask")
-			(net 42 "unconnected-(J2-BATT_B-PadB7)_2")
+			(net 44 "unconnected-(J2-BATT_B-PadB7)_1")
 			(pinfunction "BATT_B")
 			(pintype "passive+no_connect")
@@
 			(size 0.7 4.3)
 			(layers "F.Cu" "F.Mask")
-			(net 81 "unconnected-(J2-GND_B-PadA12)_4")
+			(net 87 "unconnected-(J2-GND_B-PadA12)_3")
 			(pinfunction "GND_B")
 			(pintype "passive+no_connect")
@@
 			(size 0.7 4.3)
 			(layers "F.Cu" "F.Mask")
-			(net 85 "unconnected-(J2-GND_B-PadA12)_1")
+			(net 48 "unconnected-(J2-GND_B-PadA12)_0")
 			(pinfunction "GND_B")
 			(pintype "passive+no_connect")
@@
 			(layers "F.Cu" "F.Paste" "F.Mask")
 			(roundrect_rratio 0.25)
-			(net 57 "VPT-SW")
+			(net 69 "VPT_EN")
 			(pintype "passive")
 		)
@@
 			(layers "F.Cu" "F.Paste" "F.Mask")
 			(roundrect_rratio 0.25)
-			(net 56 "VALVE2_CTRL")
+			(net 57 "SOL2_EN")
 			(pintype "passive")
 		)
@@
 			(layers "F.Cu" "F.Paste" "F.Mask")
 			(roundrect_rratio 0.25)
-			(net 55 "VALVE1_CTRL")
+			(net 56 "SOL1_EN")
 			(pintype "passive")
 		)
@@
 			(size 1.5 0.9)
 			(layers "F.Cu" "F.Paste" "F.Mask")
-			(net 55 "VALVE1_CTRL")
+			(net 56 "SOL1_EN")
 			(pinfunction "IO9")
 			(pintype "bidirectional")
@@
 			(size 1.5 0.9)
 			(layers "F.Cu" "F.Paste" "F.Mask")
-			(net 56 "VALVE2_CTRL")
+			(net 57 "SOL2_EN")
 			(pinfunction "IO10")
 			(pintype "bidirectional")
@@
 			(size 1.5 0.9)
 			(layers "F.Cu" "F.Paste" "F.Mask")
-			(net 71 "SPI_MOSI")
+			(net 81 "ADC_MOSI")
 			(pinfunction "IO12")
 			(pintype "bidirectional")
@@
 			(size 1.5 0.9)
 			(layers "F.Cu" "F.Paste" "F.Mask")
-			(net 70 "SPI_MISO")
+			(net 71 "ADC_MISO")
 			(pinfunction "IO13")
 			(pintype "bidirectional")
@@
 			(size 1.5 0.9)
 			(layers "F.Cu" "F.Paste" "F.Mask")
-			(net 69 "SPI_SCLK")
+			(net 70 "ADC_SCLK")
 			(pinfunction "IO14")
 			(pintype "bidirectional")
@@
 			(size 1.5 0.9)
 			(layers "F.Cu" "F.Paste" "F.Mask")
-			(net 57 "VPT-SW")
+			(net 69 "VPT_EN")
 			(pinfunction "IO47")
 			(pintype "bidirectional")
@@
 		(width 0.3)
 		(layer "F.Cu")
-		(net 55)
+		(net 56)
 	)
 	(segment
@@
 		(width 0.3)
 		(layer "F.Cu")
-		(net 55)
+		(net 56)
 	)
 	(segment
@@
 		(width 0.3)
 		(layer "F.Cu")
-		(net 55)
+		(net 56)
 	)
 	(segment
@@
 		(width 0.3)
 		(layer "F.Cu")
-		(net 55)
+		(net 56)
 	)
 	(segment
@@
 		(width 0.3)
 		(layer "F.Cu")
-		(net 55)
+		(net 56)
 	)
 	(segment
@@
 		(width 0.3)
 		(layer "F.Cu")
-		(net 56)
+		(net 57)
 	)
 	(segment
@@
 		(width 0.3)
 		(layer "F.Cu")
-		(net 56)
+		(net 57)
 	)
 	(segment
@@
 		(width 0.3)
 		(layer "F.Cu")
-		(net 56)
+		(net 57)
 	)
 	(segment
@@
 		(width 0.3)
 		(layer "F.Cu")
-		(net 56)
+		(net 57)
 	)
 	(segment
@@
 		(width 0.3)
 		(layer "F.Cu")
-		(net 56)
+		(net 57)
 	)
 	(segment
@@
 		(width 0.3)
 		(layer "F.Cu")
-		(net 56)
+		(net 57)
 	)
 	(segment
@@
 		(width 0.3)
 		(layer "F.Cu")
-		(net 56)
+		(net 57)
 	)
 	(segment
@@
 		(width 0.3)
 		(layer "F.Cu")
-		(net 56)
-	)
-	(segment
-		(start 129.005 99.295)
-		(end 129.005 100.75)
-		(width 0.3)
-		(layer "F.Cu")
-		(net 57)
-	)
-	(segment
-		(start 127.23 98.93)
-		(end 128.64 98.93)
-		(width 0.3)
-		(layer "F.Cu")
-		(net 57)
-	)
-	(segment
-		(start 128.64 98.93)
-		(end 129.005 99.295)
-		(width 0.3)
-		(layer "F.Cu")
 		(net 57)
 	)
@@
 	)
 	(segment
-		(start 132.2575 92.295)
-		(end 133.482106 92.295)
-		(width 0.3)
-		(layer "F.Cu")
-		(net 69)
-	)
-	(segment
-		(start 134.09 96.82)
-		(end 131.545 99.365)
-		(width 0.3)
-		(layer "F.Cu")
-		(net 69)
-	)
-	(segment
-		(start 134.09 92.902893)
-		(end 134.09 96.82)
+		(start 129.005 99.295)
+		(end 129.005 100.75)
 		(width 0.3)
 		(layer "F.Cu")
@@
 	)
 	(segment
-		(start 133.482106 92.295)
-		(end 134.09 92.902893)
+		(start 127.23 98.93)
+		(end 128.64 98.93)
 		(width 0.3)
 		(layer "F.Cu")
@@
 	)
 	(segment
-		(start 131.545 99.365)
-		(end 131.545 100.75)
+		(start 128.64 98.93)
+		(end 129.005 99.295)
 		(width 0.3)
 		(layer "F.Cu")
@@
 	)
 	(segment
-		(start 133.539212 91.645)
-		(end 134.59 92.695787)
+		(start 132.2575 92.295)
+		(end 133.482106 92.295)
 		(width 0.3)
 		(layer "F.Cu")
@@
 	)
 	(segment
-		(start 134.59 97.41)
-		(end 132.815 99.185)
+		(start 134.09 96.82)
+		(end 131.545 99.365)
 		(width 0.3)
 		(layer "F.Cu")
@@
 	)
 	(segment
-		(start 132.2575 91.645)
-		(end 133.539212 91.645)
+		(start 134.09 92.902893)
+		(end 134.09 96.82)
 		(width 0.3)
 		(layer "F.Cu")
@@
 	)
 	(segment
-		(start 134.59 92.695787)
-		(end 134.59 97.41)
+		(start 133.482106 92.295)
+		(end 134.09 92.902893)
 		(width 0.3)
 		(layer "F.Cu")
@@
 	)
 	(segment
-		(start 132.815 99.185)
-		(end 132.815 100.75)
+		(start 131.545 99.365)
+		(end 131.545 100.75)
 		(width 0.3)
 		(layer "F.Cu")
@@
 	)
 	(segment
-		(start 132.8125 91.08)
-		(end 133.681318 91.08)
+		(start 133.539212 91.645)
+		(end 134.59 92.695787)
 		(width 0.3)
 		(layer "F.Cu")
@@
 	)
 	(segment
-		(start 134.085 99.215)
-		(end 134.085 100.75)
+		(start 134.59 97.41)
+		(end 132.815 99.185)
 		(width 0.3)
 		(layer "F.Cu")
@@
 	)
 	(segment
-		(start 135.09 92.488681)
-		(end 135.09 98.21)
+		(start 132.2575 91.645)
+		(end 133.539212 91.645)
 		(width 0.3)
 		(layer "F.Cu")
@@
 	)
 	(segment
-		(start 133.681318 91.08)
-		(end 135.09 92.488681)
+		(start 134.59 92.695787)
+		(end 134.59 97.41)
 		(width 0.3)
 		(layer "F.Cu")
@@
 	)
 	(segment
-		(start 135.09 98.21)
-		(end 134.085 99.215)
+		(start 132.815 99.185)
+		(end 132.815 100.75)
 		(width 0.3)
 		(layer "F.Cu")
@@
 	)
 	(segment
+		(start 132.8125 91.08)
+		(end 133.681318 91.08)
+		(width 0.3)
+		(layer "F.Cu")
+		(net 81)
+	)
+	(segment
+		(start 134.085 99.215)
+		(end 134.085 100.75)
+		(width 0.3)
+		(layer "F.Cu")
+		(net 81)
+	)
+	(segment
+		(start 135.09 92.488681)
+		(end 135.09 98.21)
+		(width 0.3)
+		(layer "F.Cu")
+		(net 81)
+	)
+	(segment
+		(start 133.681318 91.08)
+		(end 135.09 92.488681)
+		(width 0.3)
+		(layer "F.Cu")
+		(net 81)
+	)
+	(segment
+		(start 135.09 98.21)
+		(end 134.085 99.215)
+		(width 0.3)
+		(layer "F.Cu")
+		(net 81)
+	)
+	(segment
