File: Schematics/upper_lc_board/sensing_module.kicad_sch (KiCad schematic)
At the start: 13 parts, among them J5 HALL-1, U7 ADC_ADS131M04IPWR

Commit message: add board-specifc READMEs (TODO), cleanup schematic titles
Other:
- title: Pegasus Sensing Circuitry -> Sensing Circuitry
Changed lines of the file:
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@@
 	(generator "eeschema")
 	(generator_version "8.0")
-	(paper "A4")
+	(paper "A3")
 	(title_block
-		(title "Pegasus Sensing Circuitry")
+		(title "Sensing Circuitry")
 		(company "Queen's Rocket Engineering Team")
-		(comment 1 "Upper Control Board V2")
-		(comment 2 "Jeevan Sanchez")
+		(comment 1 "Contributors: Jeevan Sanchez, Tristan Alderson")
+		(comment 2 "PEGASUS - Upper Control Board")
 	)
 	(junction
@@
 	)
 	(rectangle
-		(start 52.832 110.998)
+		(start 48.514 110.998)
 		(end 129.794 154.432)
 		(stroke
@@
 	)
 	(rectangle
-		(start 52.832 44.45)
+		(start 48.26 44.45)
 		(end 129.032 78.74)
 		(stroke
@@
 	)
 	(rectangle
-		(start 52.832 78.74)
+		(start 48.26 78.74)
 		(end 129.032 105.41)
 		(stroke
@@
 	(text "HALL Input"
 		(exclude_from_sim no)
-		(at 52.578 109.728 0)
+		(at 48.514 109.982 0)
 		(effects
 			(font
@@
 		(dnp no)
 		(property "Reference" "C13"
-			(at 57.912 57.912 0)
-			(effects
-				(font
+			(at 55.118 59.436 0)
+			(effects
+				(font

Commit message: add ed pinouts
Connections:
- net SPI_MISO renamed ADC_MISO
- net SPI_MOSI renamed ADC_MOSI
- net SPI_SCLK renamed ADC_SCLK
Changed lines of the file:
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@@
 		)
 	)
-	(global_label "SPI_MOSI"
+	(global_label "ADC_MOSI"
 		(shape input)
 		(at 213.36 77.47 0)
@@
 		)
 		(property "Intersheetrefs" "${INTERSHEET_REFS}"
-			(at 224.9933 77.47 0)
+			(at 225.5376 77.47 0)
 			(effects
 				(font
@@
 		)
 	)
-	(global_label "SPI_MISO"
+	(global_label "ADC_MISO"
 		(shape input)
 		(at 213.36 80.01 0)
@@
 		)
 		(property "Intersheetrefs" "${INTERSHEET_REFS}"
-			(at 224.9933 80.01 0)
+			(at 225.5376 80.01 0)
 			(effects
 				(font
@@
 		)
 	)
-	(global_label "SPI_SCLK"
+	(global_label "ADC_SCLK"
 		(shape input)
 		(at 213.36 74.93 0)
@@
 		)
 		(property "Intersheetrefs" "${INTERSHEET_REFS}"
-			(at 225.1747 74.93 0)
+			(at 225.719 74.93 0)
 			(effects
 				(font
