File: Schematics/upper_lc_board/modules/ESP_breakout_module/ESP_breakout_module.kicad_sch (KiCad schematic)
At the start: 24 parts, among them J8 USB_C_Female_USB2_Small, SW1 SW_ESP_BOOT_MODE, SW2 SW_ESP_RESET, U1 ESP32-S3-WROOM-1-N16, U2 ISO1044BDR

Commit message: organizational work
Parts:
- C1: JLCPCB (none) -> C15849
- C2, C4, C5, C6, C7: JLCPCB (none) -> C14663
Changed lines of the file:
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@@
+			)
+		)
+		(property "JLCPCB" "C14663"
+			(at 105.41 55.88 0)
+			(effects
+				(font
+					(size 1.27 1.27)
+				)
+				(hide yes)
 			)
 		)
@@
 		)
 		(property "LCSC" "C14663"
+			(at 228.6 48.26 0)
+			(effects
+				(font
+					(size 1.27 1.27)
+				)
+				(hide yes)
+			)
+		)
+		(property "JLCPCB" "C14663"
 			(at 228.6 48.26 0)
 			(effects
@@
 			)
 		)
+		(property "JLCPCB" "C14663"
+			(at 161.29 66.04 0)
+			(effects
+				(font
+					(size 1.27 1.27)
+				)
+				(hide yes)
+			)
+		)
 		(pin "1"
 		)
@@
 			)
 		)
+		(property "JLCPCB" "C15849"
+			(at 62.23 69.85 0)
+			(effects
+				(font
+					(size 1.27 1.27)
+				)
+				(hide yes)
+			)
+		)
 		(pin "2"
 		)
@@
 			)
 		)
+		(property "JLCPCB" "C14663"
+			(at 203.2 48.26 0)
+			(effects
+				(font
+					(size 1.27 1.27)
+				)
+				(hide yes)
+			)
+		)
 		(pin "2"
 		)
@@
 			(at 161.29 48.26 0)
 			(effects
+				(font
+					(size 1.27 1.27)
+				)
+				(hide yes)
+			)
+		)
+		(property "JLCPCB" "C14663"
+			(at 161.29 48.26 0)
+			(effects

Commit message: more organizational work, add shared footprint, model, symbol dirs and clean up individuals
Other:
- title: ULC Board ESP32-S3 Breakout Circuitry  -> PHEONIX | ESP32-S3 Breakout Circuitry
Changed lines of the file:
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@@
 	(paper "A4")
 	(title_block
-		(title "ULC Board ESP32-S3 Breakout Circuitry ")
+		(title "PHEONIX | ESP32-S3 Breakout Circuitry")
 		(rev "A")
 		(company "Queen's Rocket Engineering Team")
@@
 			)
 		)
-		(property "Datasheet" "${KIPRJMOD}/../../Datasheets/USBSC-conn.pdf"
+		(property "Datasheet" "${KIPRJMOD}/../../Documentation/USBconn_DS.pdf"
 			(at 154.94 113.03 0)
 			(effects
@@
 			)
 		)
-		(property "Datasheet" "${KIPRJMOD}/../../Datasheets/MCU-esp32-s3-wroom-1_wroom-1u_datasheet_en.pdf"
+		(property "Datasheet" "${KIPRJMOD}/../../Documentation/mcu_ESP32-S3-WROOM-1-N16_DS.pdf"
 			(at 92.71 88.9 0)
 			(effects
@@
 			)
 		)
-		(property "Datasheet" "${KIPRJMOD}/../../Datasheets/LED-WS2812B.pdf"
+		(property "Datasheet" "${KIPRJMOD}/../../Documentation/LED_WS2812B_DS.pdf"
 			(at 119.38 169.545 0)
 			(effects
@@
 			)
 		)
-		(property "Datasheet" "${KIPRJMOD}/../../Datasheets/buttons-modeselec.pdf"
+		(property "Datasheet" "${KIPRJMOD}/../../Documentation/button_C318884_DS.pdf"
 			(at 156.21 39.37 0)
 			(effects
@@
 			)
 		)
-		(property "Datasheet" "${KIPRJMOD}/../../Datasheets/CAN-T_ISO1044.pdf"
+		(property "Datasheet" "${KIPRJMOD}/../../Documentation/CANT_ISO1044_DS.pdf"
 			(at 215.9 67.31 0)
 			(effects
@@
 			)
 		)
-		(property "Datasheet" "${KIPRJMOD}/../../Datasheets/buttons-modeselec.pdf"
+		(property "Datasheet" "${KIPRJMOD}/../../Documentation/button_C318884_DS.pdf"
 			(at 156.21 57.15 0)
 			(effects
