File: Schematics/upper_lc_board/modules/sensor_module/sensor_module.kicad_sch (KiCad schematic)
At the start: 22 parts, among them J5 HALL, U7 ADC_ADS131M04IPWR

Commit message: organizational work
Parts:
- removed C34: 1uF_10V, Capacitor_SMD:C_1206_3216Metric, symbol Device:C
- C21, C23: JLCPCB (none) -> C15849
- C33: value 0.1uF_10V -> 0.1uF; footprint Capacitor_SMD:C_0805_2012Metric -> Capacitor_SMD:C_0603_1608Metric; JLCPCB (none) -> C14663
Connections:
- net GND: no longer C21.1, C22.2, R21.1, R23.1, U7.10 (AIN3P), U7.2 (AGND), U7.9 (AIN3N)
- new net GNDA: C21.1, C22.2, R21.1, R23.1, U7.10 (AIN3P), U7.2 (AGND), U7.9 (AIN3N)
Other:
- moved on the sheet: C17, C18, C19, C21, C22, C23, C33, D10, D11, D12, D13, J5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

Commit message: more organizational work, add shared footprint, model, symbol dirs and clean up individuals
Other:
- title: ULC Board Sensor Circuitry -> PHEONIX | Sensor Circuitry
Changed lines of the file:
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@@
 	(paper "A4")
 	(title_block
-		(title "ULC Board Sensor Circuitry")
+		(title "PHEONIX | Sensor Circuitry")
 		(rev "A")
 		(company "Queen's Rocket Engineering Team")
@@
 			)
 		)
-		(property "Datasheet" "${KIPRJMOD}/../../Datasheets/ADC-ads131m04.pdf"
+		(property "Datasheet" "${KIPRJMOD}/../../Documentation/ADC_ads131m04_DS.pdf"
 			(at 170.18 69.85 0)
 			(effects
@@
 			)
 		)
-		(property "Datasheet" "${KIPRJMOD}/../../Datasheets/CONN-530470460.pdf"
+		(property "Datasheet" "${KIPRJMOD}/../../Documentation/conn_m_530470460.pdf"
 			(at 53.34 128.27 0)
 			(effects
