File: Schematics/upper_lc_board/modules/solenoid_module/solenoid_module.kicad_sch (KiCad schematic)
At the start: 6 parts

Commit message: more organizational work, add shared footprint, model, symbol dirs and clean up individuals
Other:
- title: ULC Board Solenoid Driver Circuitry -> PHEONIX | Actuation Circuitry
Changed lines of the file:
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@@
 	(paper "A4")
 	(title_block
-		(title "ULC Board Solenoid Driver Circuitry")
+		(title "PHEONIX | Actuation Circuitry")
 		(rev "A")
 		(company "Queen's Rocket Engineering Team")
