File: Schematics/lower_lc_board/modules/actuation_module/actuation_module.kicad_sch (KiCad schematic)
At the start: 13 parts, among them Q5 2N7002, U12 DMP4065S-7

Commit message: pcb design
Parts:
- U12: footprint ul_SI2301CDS-T1-GE3:TO-236_VIS -> Package_TO_SOT_SMD:SOT-23
Changed lines of the file:
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@@
 			)
 		)
-		(property "Footprint" "ul_SI2301CDS-T1-GE3:TO-236_VIS"
+		(property "Footprint" "Package_TO_SOT_SMD:SOT-23"
 			(at 82.55 125.73 0)
 			(effects
