File: Schematics/lower_lc_board/modules/actuation_module/actuation_module.kicad_sch (KiCad schematic)
At the start: 13 parts, among them Q5 2N7002, U12 DMP4065S-7

Commit message: increase width on power rails from USB and SWD, start tuning diff pairs
Parts:
- C46: Digikey 732-8419-1-ND -> 732-8511-1-ND; JLCPCB 865080545012 -> (none)
- D11, D12: JLCPCB (none) -> C2290
- R30, R31: Digikey 311-4.70KFRCT-ND -> (none)
- R52: JLCPCB (none) -> C25804
- R53: JLCPCB (none) -> C8218
- U12: Digikey (none) -> C182476
Changed lines of the file:
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@@
 			)
 		)
-		(property "Digikey" "732-8419-1-ND"
+		(property "Digikey" "732-8511-1-ND"
 			(at 229.87 55.88 0)
 			(effects
@@
 			)
 		)
-		(property "JLCPCB" "865080545012"
+		(property "JLCPCB" ""
 			(at 229.87 55.88 0)
 			(effects
@@
 			)
 		)
-		(property "Digikey" "311-4.70KFRCT-ND"
+		(property "Digikey" ""
 			(at 102.87 76.2 90)
 			(effects
@@
 			)
 		)
+		(property "JLCPCB" "C25804"
+			(at 87.63 114.3 0)
+			(effects
+				(font
+					(size 1.27 1.27)
+				)
+				(hide yes)
+			)
+		)
 		(pin "1"
 		)
@@
 			)
 		)
+		(property "JLCPCB" "C8218"
+			(at 93.98 110.49 0)
+			(effects
+				(font
+					(size 1.27 1.27)
+				)
+				(hide yes)
+			)
+		)
 		(pin "1"
 		)
@@
 		)
 		(property "Description" ""
+			(at 82.55 125.73 0)
+			(effects
+				(font
+					(size 1.27 1.27)
+				)
+				(hide yes)
+			)
+		)
+		(property "Digikey" "C182476"
 			(at 82.55 125.73 0)
 			(effects
@@
 			)
 		)
-		(property "Digikey" "311-4.70KFRCT-ND"
+		(property "Digikey" ""
 			(at 102.87 60.96 90)
 			(effects
@@
 			)
 		)
+		(property "JLCPCB" "C2290"
+			(at 95.25 76.2 0)
+			(effects
+				(font
+					(size 1.27 1.27)
+				)
+				(hide yes)
+			)
+		)
 		(pin "1"
 		)
@@
 			(at 95.25 60.96 0)
 			(effects
+				(font
+					(size 1.27 1.27)
+				)
+				(hide yes)
+			)
+		)
+		(property "JLCPCB" "C2290"
+			(at 95.25 60.96 0)
+			(effects
