File: Schematics/lower_lc_board/modules/sensing_module/sensing_module.kicad_sch (KiCad schematic)
At the start: 26 parts, among them J4 HALL-1, J5 HALL-2, Q3 2N7002, U11 SI2301CDS-T1-GE3, U9 ADC_ADS131M04IPWR

Commit message: adjust routing for 0603 min. footprints
Parts:
- C25, C26, C27, C56: JLCPCB C57112 -> (none)
- C29: footprint Capacitor_SMD:C_0402_1005Metric -> Capacitor_SMD:C_0603_1608Metric
- R17, R18, R19, R20: footprint Resistor_SMD:R_0402_1005Metric -> Resistor_SMD:R_0603_1608Metric
Connections:
- net TC_N_CLAMPED_1: now also C56.1, U9.9 (AIN3N); no longer C25.1, U9.8 (AIN2N)
- net TC_N_CLAMPED_2: now also C25.1, U9.8 (AIN2N); no longer C56.1, U9.9 (AIN3N)
- net TC_P_CLAMPED_1: now also C56.2, U9.10 (AIN3P); no longer C25.2, U9.7 (AIN2P)
- net TC_P_CLAMPED_2: now also C25.2, U9.7 (AIN2P); no longer C56.2, U9.10 (AIN3P)
Changed lines of the file:
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@@
 		)
 	)
-	(label "TC_N_CLAMPED_1"
-		(at 127 67.31 180)
+	(label "TC_N_2"
+		(at 218.44 113.03 180)
 		(fields_autoplaced yes)
 		(effects
@@
 		)
 	)
-	(label "TC_N_2"
-		(at 218.44 113.03 180)
+	(label "TC_N_CLAMPED_2"
+		(at 127 67.31 180)
 		(fields_autoplaced yes)
 		(effects
@@
 	)
 	(label "TC_P_CLAMPED_2"
-		(at 127 83.82 180)
+		(at 127 73.66 180)
 		(fields_autoplaced yes)
 		(effects
@@
 		)
 	)
-	(label "TC_N_CLAMPED_2"
+	(label "TC_N_CLAMPED_1"
 		(at 127 77.47 180)
 		(fields_autoplaced yes)
@@
 		)
 	)
-	(label "TC_P_CLAMPED_1"
-		(at 127 73.66 180)
-		(fields_autoplaced yes)
-		(effects
-			(font
-				(size 1.27 1.27)
-			)
-			(justify right bottom)
-		)
-	)
 	(label "PT1"
 		(at 49.53 44.45 180)
@@
 		)
 	)
+	(label "TC_P_CLAMPED_1"
+		(at 127 83.82 180)
+		(fields_autoplaced yes)
+		(effects
+			(font
+				(size 1.27 1.27)
+			)
+			(justify right bottom)
+		)
+	)
 	(global_label "VPT-SW"
 		(shape input)
@@
 			)
 		)
-		(property "JLCPCB" "C57112"
+		(property "JLCPCB" ""
 			(at 135.89 80.01 0)
 			(effects
@@
 			)
 		)
-		(property "Footprint" "Resistor_SMD:R_0402_1005Metric"
+		(property "Footprint" "Resistor_SMD:R_0603_1608Metric"
 			(at 127 44.958 90)
 			(effects
@@
 			)
 		)
-		(property "JLCPCB" "C57112"
+		(property "JLCPCB" ""
 			(at 134.62 60.96 0)
 			(effects
@@
 			)
 		)
-		(property "Footprint" "Resistor_SMD:R_0402_1005Metric"
+		(property "Footprint" "Resistor_SMD:R_0603_1608Metric"
 			(at 89.662 128.27 90)
 			(effects
@@
 			)
 		)
-		(property "Footprint" "Resistor_SMD:R_0402_1005Metric"
+		(property "Footprint" "Resistor_SMD:R_0603_1608Metric"
 			(at 128.27 58.928 90)
 			(effects
@@
 			)
 		)
-		(property "JLCPCB" "C57112"
+		(property "JLCPCB" ""
 			(at 134.62 69.85 0)
 			(effects
@@
 			)
 		)
-		(property "Footprint" "Capacitor_SMD:C_0402_1005Metric"
+		(property "Footprint" "Capacitor_SMD:C_0603_1608Metric"
 			(at 190.5 73.9648 0)
 			(effects
@@
 			)
 		)
-		(property "JLCPCB" "C57112"
+		(property "JLCPCB" ""
 			(at 133.35 46.99 0)
 			(effects
@@
 			)
 		)
-		(property "Footprint" "Resistor_SMD:R_0402_1005Metric"
+		(property "Footprint" "Resistor_SMD:R_0603_1608Metric"
 			(at 93.218 144.78 90)
 			(effects

Commit message: more local pours and 0402 adjustments
Parts:
- R22, R44, R49: footprint Resistor_SMD:R_0402_1005Metric -> Resistor_SMD:R_0603_1608Metric
- R23: footprint Resistor_SMD:R_0402_1005Metric -> Resistor_SMD:R_0805_2012Metric
- TH1: footprint Resistor_SMD:R_0402_1005Metric -> Resistor_SMD:R_0603_1608Metric; Digikey 273-TX06F103F3435ERCT-ND -> P60.4DBCT-ND
Changed lines of the file:
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@@
 			)
 		)
-		(property "Footprint" "Resistor_SMD:R_0402_1005Metric"
+		(property "Footprint" "Resistor_SMD:R_0805_2012Metric"
 			(at 228.6 75.438 90)
 			(effects
@@
 			)
 		)
-		(property "Footprint" "Resistor_SMD:R_0402_1005Metric"
+		(property "Footprint" "Resistor_SMD:R_0603_1608Metric"
 			(at 241.3 62.992 90)
 			(effects
@@
 			)
 		)
-		(property "Footprint" "Resistor_SMD:R_0402_1005Metric"
+		(property "Footprint" "Resistor_SMD:R_0603_1608Metric"
 			(at 133.35 184.15 0)
 			(effects
@@
 			)
 		)
-		(property "Digikey" "273-TX06F103F3435ERCT-ND"
+		(property "Digikey" "P60.4DBCT-ND"
 			(at 133.35 184.15 0)
 			(effects
@@
 			)
 		)
-		(property "Footprint" "Resistor_SMD:R_0402_1005Metric"
+		(property "Footprint" "Resistor_SMD:R_0603_1608Metric"
 			(at 204.978 82.55 90)
 			(effects
@@
 			)
 		)
-		(property "Footprint" "Resistor_SMD:R_0402_1005Metric"
+		(property "Footprint" "Resistor_SMD:R_0603_1608Metric"
 			(at 218.44 75.438 90)
 			(effects

Commit message: review of schematics and pcb
- verified all STM pins
- reviewed all circuits
- reviewed trace clearences, made sure routes are connected, etc.
Parts:
- C35: JLCPCB (none) -> C13585
- J4, J5: Digikey 900-0530470460-ND -> 455-S04B-PASK-2-ND
- Q3: JLCPCB (none) -> C8545
- R22: JLCPCB C25744 -> C25804
- R23: value 10k -> 4.7K; JLCPCB C25744 -> C23162
- U11: value SI2301CDS-T1-GE3 -> DMP4065S-7
Other:
- note added: "CJC"
- moved on the sheet: R25, TH1
Changed lines of the file:
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@@
 	)
 	(junction
-		(at 133.35 177.8)
-		(diameter 0)
-		(color 0 0 0 0)
-	)
-	(junction
 		(at 222.758 121.92)
 		(diameter 0)
@@
 	)
 	(junction
-		(at 133.35 167.64)
+		(at 123.19 177.8)
+		(diameter 0)
+		(color 0 0 0 0)
+	)
+	(junction
+		(at 114.3 177.8)
 		(diameter 0)
 		(color 0 0 0 0)
@@
 	(wire
 		(pts
-			(xy 133.35 175.26) (xy 133.35 177.8)
+			(xy 123.19 177.8) (xy 125.73 177.8)
+		)
+		(stroke
+			(width 0)
+			(type default)
+		)
+	)
+	(wire
+		(pts
+			(xy 121.92 177.8) (xy 123.19 177.8)
 		)
 		(stroke
@@
 	(wire
 		(pts
-			(xy 133.35 177.8) (xy 137.16 177.8)
+			(xy 123.19 177.8) (xy 123.19 170.18)
 		)
 		(stroke
@@
 	(wire
 		(pts
-			(xy 133.35 177.8) (xy 133.35 179.07)
-		)
-		(stroke
-			(width 0)
-			(type default)
-		)
-	)
-	(wire
-		(pts
 			(xy 49.53 54.61) (xy 52.07 54.61)
 		)
@@
 		)
 	)
+	(rectangle
+		(start 107.188 163.322)
+		(end 145.542 186.436)
+		(stroke
+			(width 0)
+			(type default)
+			(color 0 0 0 1)
+		)
+		(fill
+			(type none)
+		)
+	)
 	(text "Vf = 1.25v (at 100ma),\nVmax = 3.3+1.25,\n0.95v/5ma ~ 200ohms current limiter"
 		(exclude_from_sim no)
@@
 	(text "place as close as possible to thermocouple input\nfor CJC measuring accuracy"
 		(exclude_from_sim no)
-		(at 133.35 163.322 0)
+		(at 120.142 165.354 0)
+		(effects
+			(font
+				(size 0.635 0.635)
+				(color 0 0 0 1)
+			)
+		)
+	)
+	(text "CJC"
+		(exclude_from_sim no)
+		(at 107.188 162.052 0)
 		(effects
 			(font
 				(size 1.27 1.27)
+				(thickness 0.254)
+				(bold yes)
+				(italic yes)
 				(color 0 0 0 1)
 			)
+			(justify left)
 		)
 	)
@@
 	(global_label "TEMP_SENSE"
 		(shape input)
-		(at 137.16 177.8 0)
+		(at 123.19 170.18 0)
 		(fields_autoplaced yes)
 		(effects
@@
 		)
 		(property "Intersheetrefs" "${INTERSHEET_REFS}"
-			(at 151.9983 177.8 0)
+			(at 138.0283 170.18 0)
 			(effects
 				(font
@@
 			)
 		)
+		(property "JLCPCB" "C8545"
+			(at 223.52 59.69 0)
+			(effects
+				(font
+					(size 1.27 1.27)
+				)
+				(hide yes)
+			)
+		)
 		(pin "1"
 		)
@@
 			)
 		)
-		(property "Value" "10k"
+		(property "Value" "4.7K"
 			(at 230.378 73.66 90)
 			(effects
@@
 			)
 		)
-		(property "JLCPCB" "C25744"
+		(property "JLCPCB" "C23162"
 			(at 228.6 73.66 0)
 			(effects
@@
 			)
 		)
-		(property "Digikey" "900-0530470460-ND"
+		(property "Digikey" "455-S04B-PASK-2-ND"
 			(at 49.53 154.94 90)
 			(effects
@@
 	(symbol
 		(lib_id "power:+3V3")
-		(at 133.35 167.64 90)
+		(at 114.3 177.8 180)
 		(unit 1)
 		(exclude_from_sim no)
@@
 		(on_board yes)
 		(dnp no)
-		(fields_autoplaced yes)
 		(property "Reference" "#PWR074"
-			(at 137.16 167.64 0)
+			(at 114.3 173.99 0)
 			(effects
 				(font
@@
 		)
 		(property "Value" "+3V3"
-			(at 129.54 167.6399 90)
+			(at 116.84 181.864 0)
 			(effects
 				(font
@@
 		)
 		(property "Footprint" ""
-			(at 133.35 167.64 0)
+			(at 114.3 177.8 0)
 			(effects
 				(font
@@
 		)
 		(property "Datasheet" ""
-			(at 133.35 167.64 0)
+			(at 114.3 177.8 0)
 			(effects
 				(font
@@
 		)
 		(property "Description" "Power symbol creates a global label with name \"+3V3\""
-			(at 133.35 167.64 0)
+			(at 114.3 177.8 0)
 			(effects
 				(font
@@
 	(symbol
 		(lib_id "Device:R")
-		(at 133.35 171.45 180)
+		(at 118.11 177.8 270)
 		(unit 1)
 		(exclude_from_sim no)
@@
 		(dnp no)
 		(property "Reference" "R25"
-			(at 135.89 170.1799 0)
+			(at 119.634 175.514 90)
 			(effects
 				(font
@@
 		)
 		(property "Value" "10k"
-			(at 133.35 172.72 90)
+			(at 119.38 177.8 90)
 			(effects
 				(font
@@
 		)
 		(property "Footprint" "Resistor_SMD:R_0603_1608Metric"
-			(at 135.128 171.45 90)
+			(at 118.11 176.022 90)
 			(effects
 				(font
@@
 		)
 		(property "Datasheet" "~"
-			(at 133.35 171.45 0)
+			(at 118.11 177.8 0)
 			(effects
 				(font
@@
 		)
 		(property "Description" "Resistor"
-			(at 133.35 171.45 0)
+			(at 118.11 177.8 0)
 			(effects
 				(font
@@
 		)
 		(property "LCSC" "C25804"
-			(at 133.35 171.45 0)
+			(at 118.11 177.8 0)
 			(effects
 				(font
@@
 	(symbol
 		(lib_id "power:+3V3")
-		(at 133.35 167.64 90)
+		(at 114.3 177.8 180)
 		(unit 1)
 		(exclude_from_sim no)
@@
 		(on_board yes)
 		(dnp no)
-		(fields_autoplaced yes)
 		(property "Reference" "#PWR082"
-			(at 137.16 167.64 0)
+			(at 114.3 173.99 0)
 			(effects
 				(font
@@
 		)
 		(property "Value" "+3V3"
-			(at 129.54 167.6399 90)
+			(at 116.84 181.864 0)
 			(effects
 				(font
@@
 		)
 		(property "Footprint" ""
-			(at 133.35 167.64 0)
+			(at 114.3 177.8 0)
 			(effects
 				(font
@@
 		)
 		(property "Datasheet" ""
-			(at 133.35 167.64 0)
+			(at 114.3 177.8 0)
 			(effects
 				(font
@@
 		)
 		(property "Description" "Power symbol creates a global label with name \"+3V3\""
-			(at 133.35 167.64 0)
+			(at 114.3 177.8 0)
 			(effects
 				(font
@@
 	(symbol
 		(lib_id "power:GND")
-		(at 133.35 189.23 0)
+		(at 135.89 177.8 90)
 		(unit 1)
 		(exclude_from_sim no)
@@
 		(fields_autoplaced yes)
 		(property "Reference" "#PWR083"
-			(at 133.35 195.58 0)
+			(at 142.24 177.8 0)
 			(effects
 				(font
@@
 		)
 		(property "Value" "GND"
-			(at 133.35 194.31 0)
+			(at 140.97 177.8 0)
 			(effects
 				(font
@@
 		)
 		(property "Footprint" ""
-			(at 133.35 189.23 0)
+			(at 135.89 177.8 0)
 			(effects
 				(font
@@
 		)
 		(property "Datasheet" "https://www.ti.com/lit/ds/symlink/drv5055.pdf?HQS=dis-dk-null-digikeymode-dsf-pf-null-wwe&ts=1641231273160"
-			(at 133.35 189.23 0)
+			(at 135.89 177.8 0)
 			(effects
 				(font
@@
 		)
 		(property "Description" "Hall effect sensor."
-			(at 133.35 189.23 0)
+			(at 135.89 177.8 0)
 			(effects
 				(font
@@
 	(symbol
 		(lib_id "Device:Thermistor")
-		(at 133.35 184.15 0)
+		(at 130.81 177.8 90)
 		(unit 1)
 		(exclude_from_sim no)
@@
 		(dnp no)
 		(property "Reference" "TH1"
-			(at 121.412 182.88 0)
+			(at 134.366 180.848 90)
 			(effects
 				(font
@@
 		)
 		(property "Value" "Thermistor"
-			(at 121.412 185.42 0)
+			(at 134.366 183.388 90)
 			(effects
 				(font
@@
 		)
 		(property "Footprint" "Resistor_SMD:R_0603_1608Metric"
-			(at 133.35 184.15 0)
+			(at 130.81 177.8 0)
 			(effects
 				(font
@@
 		)
 		(property "Datasheet" "${KIPRJMOD}/../../Documentation/thermistor_tx_DS.pdf"
-			(at 133.35 184.15 0)
+			(at 130.81 177.8 0)
 			(effects
 				(font
@@
 		)
 		(property "Description" "Temperature dependent resistor for CJC, *place as close to TC connector as possible. *will need conditoning in code (averaging)"
-			(at 133.35 184.15 0)
+			(at 130.81 177.8 0)
 			(effects
 				(font
@@
 		)
 		(property "Digikey" "P60.4DBCT-ND"
-			(at 133.35 184.15 0)
+			(at 130.81 177.8 0)
 			(effects
 				(font
@@
 		)
 		(property "Model" "TX06F103F3435ER"
-			(at 133.35 184.15 0)
+			(at 130.81 177.8 0)
 			(effects
 				(font
@@
 			)
 		)
-		(property "Value" "SI2301CDS-T1-GE3"
+		(property "Value" "DMP4065S-7"
 			(at 253.746 75.946 0)
 			(effects
@@
 			)
 		)
-		(property "Datasheet" "${KIPRJMOD}/../../Documentation/pmosfet_si2301cd_DS.pdf"
+		(property "Datasheet" "${KIPRJMOD}/../../Documentation/pmosfet_DMP4065S-7_DS.pdf"
 			(at 229.87 80.01 0)
 			(effects
@@
 			)
 		)
-		(property "Digikey" "900-0530470460-ND"
+		(property "Digikey" "455-S04B-PASK-2-ND"
 			(at 49.53 115.57 90)
 			(effects
@@
 			)
 		)
-		(property "JLCPCB" "C25744"
+		(property "JLCPCB" "C25804"
 			(at 218.44 73.66 0)
 			(effects
@@
 			(at 100.33 44.45 0)
 			(effects
+				(font
+					(size 1.27 1.27)
+				)
+				(hide yes)
+			)
+		)
+		(property "JLCPCB" "C13585"
+			(at 100.33 44.45 0)
+			(effects

Commit message: pcb design
Parts:
- U11: footprint ul_SI2301CDS-T1-GE3:TO-236_VIS -> Package_TO_SOT_SMD:SOT-23
Changed lines of the file:
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@@
 			)
 		)
-		(property "Footprint" "ul_SI2301CDS-T1-GE3:TO-236_VIS"
+		(property "Footprint" "Package_TO_SOT_SMD:SOT-23"
 			(at 229.87 80.01 0)
 			(effects
