File: Schematics/upper_lc_board_v2/modules/power_module/power_module.kicad_sch (KiCad schematic)
At the start: 42 parts, among them J2 Stack Male Edge Connector, Q1 2N7002, Q5 2N7002, U3 AMS1117, U4 ID_LM66100DCKR, U5 ID_LM66100DCKR, U6 DMP4065S-7, U9 DMP4065S-7

Commit message: pcb design
Parts:
- U6, U9: footprint ul_SI2301CDS-T1-GE3:TO-236_VIS -> Package_TO_SOT_SMD:SOT-23
Changed lines of the file:
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@@
 	)
 	(junction
-		(at 80.01 43.18)
-		(diameter 0)
-		(color 194 0 0 1)
-	)
-	(junction
 		(at 134.62 138.43)
 		(diameter 0)
@@
 	)
 	(junction
+		(at 80.01 43.18)
+		(diameter 0)
+		(color 0 0 0 0)
+	)
+	(junction
 		(at 179.07 66.04)
 		(diameter 0)
@@
 	)
 	(symbol
+		(lib_id "EdgeConnectorV2:Stack Male Edge Connector")
+		(at 66.04 62.23 0)
+		(unit 1)
+		(exclude_from_sim no)
+		(in_bom yes)
+		(on_board yes)
+		(dnp no)
+		(fields_autoplaced yes)
+		(property "Reference" "J2"
+			(at 66.04 35.56 0)
+			(effects
+				(font
+					(size 1.27 1.27)
+				)
+			)
+		)
+		(property "Value" "Stack Male Edge Connector"
+			(at 66.04 38.1 0)
+			(effects
+				(font
+					(size 1.27 1.27)
+				)
+			)
+		)
+		(property "Footprint" "Connector_PCBEdge:BUS_PCIexpress_x1"
+			(at 66.04 85.09 0)
+			(effects
+				(font
+					(size 1.27 1.27)
+				)
+				(hide yes)
+			)
+		)
+		(property "Datasheet" ""
+			(at 60.706 81.28 0)
+			(effects
+				(font
+					(size 1.27 1.27)
+				)
+				(hide yes)
+			)
+		)
+		(property "Description" "QRET SRAD Male Stack Edge Connector (PCIe x1 Connector). Generation 2"
+			(at 62.23 57.912 0)
+			(effects
+				(font
+					(size 1.27 1.27)
+				)
+				(hide yes)
+			)
+		)
+		(pin "B3"
+		)
+		(pin "A10"
+		)
+		(pin "A3"
+		)
+		(pin "B4"
+		)
+		(pin "B10"
+		)
+		(pin "A17"
+		)
+		(pin "B13"
+		)
+		(pin "A1"
+		)
+		(pin "A11"
+		)
+		(pin "A14"
+		)
+		(pin "A15"
+		)
+		(pin "A7"
+		)
+		(pin "B12"
+		)
+		(pin "B16"
+		)
+		(pin "B14"
+		)
+		(pin "A13"
+		)
+		(pin "A16"
+		)
+		(pin "B11"
+		)
+		(pin "A18"
+		)
+		(pin "A2"
+		)
+		(pin "B15"
+		)
+		(pin "B1"
+		)
+		(pin "A6"
+		)
+		(pin "B17"
+		)
+		(pin "B18"
+		)
+		(pin "B5"
+		)
+		(pin "A9"
+		)
+		(pin "B6"
+		)
+		(pin "A5"
+		)
+		(pin "B2"
+		)
+		(pin "A4"
+		)
+		(pin "B7"
+		)
+		(pin "B8"
+		)
+		(pin "B9"
+		)
+		(pin "A8"
+		)
+		(pin "A12"
+		)
+		(instances
+			(project "upper_lc_board_v2"
+				(path "/8de962ac-ee95-4233-a205-efbcd04063bc/94566a7d-86bb-4a04-89fe-f21a893d6a23"
+					(reference "J2")
+					(unit 1)
+				)
+			)
+		)
+	)
+	(symbol
 		(lib_id "QRET_Buck_PSU:LM66100DCKR")
 		(at 151.13 53.34 0)
@@
 	)
 	(symbol
-		(lib_id "EdgeConnectorV2:Stack Male Edge Connector")
-		(at 66.04 62.23 0)
-		(unit 1)
-		(exclude_from_sim no)
-		(in_bom yes)
-		(on_board yes)
-		(dnp no)
-		(property "Reference" "J2"
-			(at 66.04 35.56 0)
-			(effects
-				(font
-					(size 1.27 1.27)
-				)
-			)
-		)
-		(property "Value" "Stack Male Edge Connector"
-			(at 66.04 38.1 0)
-			(effects
-				(font
-					(size 1.27 1.27)
-				)
-			)
-		)
-		(property "Footprint" "Connector_PCBEdge:BUS_PCIexpress_x1"
-			(at 66.04 85.09 0)
-			(effects
-				(font
-					(size 1.27 1.27)
-				)
-				(hide yes)
-			)
-		)
-		(property "Datasheet" ""
-			(at 60.706 81.28 0)
-			(effects
-				(font
-					(size 1.27 1.27)
-				)
-				(hide yes)
-			)
-		)
-		(property "Description" "QRET SRAD Male Stack Edge Connector (PCIe x1 Connector). Generation 2"
-			(at 62.23 57.912 0)
-			(effects
-				(font
-					(size 1.27 1.27)
-				)
-				(hide yes)
-			)
-		)
-		(pin "B3"
-		)
-		(pin "A10"
-		)
-		(pin "A3"
-		)
-		(pin "B4"
-		)
-		(pin "B10"
-		)
-		(pin "A17"
-		)
-		(pin "B13"
-		)
-		(pin "A1"
-		)
-		(pin "A11"
-		)
-		(pin "A14"
-		)
-		(pin "A15"
-		)
-		(pin "A7"
-		)
-		(pin "B12"
-		)
-		(pin "B16"
-		)
-		(pin "B14"
-		)
-		(pin "A13"
-		)
-		(pin "A16"
-		)
-		(pin "B11"
-		)
-		(pin "A18"
-		)
-		(pin "A2"
-		)
-		(pin "B15"
-		)
-		(pin "B1"
-		)
-		(pin "A6"
-		)
-		(pin "B17"
-		)
-		(pin "B18"
-		)
-		(pin "B5"
-		)
-		(pin "A9"
-		)
-		(pin "B6"
-		)
-		(pin "A5"
-		)
-		(pin "B2"
-		)
-		(pin "A4"
-		)
-		(pin "B7"
-		)
-		(pin "B8"
-		)
-		(pin "B9"
-		)
-		(pin "A8"
-		)
-		(pin "A12"
-		)
-		(instances
-			(project "upper_lc_board_v2"
-				(path "/8de962ac-ee95-4233-a205-efbcd04063bc/94566a7d-86bb-4a04-89fe-f21a893d6a23"
-					(reference "J2")
-					(unit 1)
-				)
-			)
-		)
-	)
-	(symbol
 		(lib_id "power:PWR_FLAG")
 		(at 163.83 137.16 0)
@@
 			)
 		)
-		(property "Footprint" "ul_SI2301CDS-T1-GE3:TO-236_VIS"
+		(property "Footprint" "Package_TO_SOT_SMD:SOT-23"
 			(at 217.17 111.76 0)
 			(effects
@@
 			)
 		)
-		(property "Footprint" "ul_SI2301CDS-T1-GE3:TO-236_VIS"
+		(property "Footprint" "Package_TO_SOT_SMD:SOT-23"
 			(at 217.17 60.96 0)
 			(effects

Commit message: add additional LEDs
Parts:
- added TP11: 24V-TP-H, TestPoint:TestPoint_THTPad_D1.0mm_Drill0.5mm, symbol Connector:TestPoint
- TP3: value 24V-TP -> 24V-TP-P; footprint TestPoint:TestPoint_Pad_D1.0mm -> TestPoint:TestPoint_Pad_1.5x1.5mm
Connections:
- net +24V: now also TP11.1
Changed lines of the file:
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@@
 	)
 	(symbol
+		(lib_id "Connector:TestPoint")
+		(at 27.94 135.89 0)
+		(unit 1)
+		(exclude_from_sim no)
+		(in_bom yes)
+		(on_board yes)
+		(dnp no)
+		(property "Reference" "TP11"
+			(at 29.464 129.794 0)
+			(effects
+				(font
+					(size 1.27 1.27)
+				)
+				(justify left)
+			)
+		)
+		(property "Value" "24V-TP-H"
+			(at 29.21 132.08 0)
+			(effects
+				(font
+					(size 1.27 1.27)
+				)
+				(justify left)
+			)
+		)
+		(property "Footprint" "TestPoint:TestPoint_THTPad_D1.0mm_Drill0.5mm"
+			(at 33.02 135.89 0)
+			(effects
+				(font
+					(size 1.27 1.27)
+				)
+				(hide yes)
+			)
+		)
+		(property "Datasheet" "~"
+			(at 33.02 135.89 0)
+			(effects
+				(font
+					(size 1.27 1.27)
+				)
+				(hide yes)
+			)
+		)
+		(property "Description" "test point"
+			(at 27.94 135.89 0)
+			(effects
+				(font
+					(size 1.27 1.27)
+				)
+				(hide yes)
+			)
+		)
+		(pin "1"
+		)
+		(instances
+			(project "upper_lc_board_v2"
+				(path "/8de962ac-ee95-4233-a205-efbcd04063bc/94566a7d-86bb-4a04-89fe-f21a893d6a23"
+					(reference "TP11")
+					(unit 1)
+				)
+			)
+		)
+	)
+	(symbol
 		(lib_id "Device:R")
 		(at 43.18 106.68 0)
@@
 	)
 	(symbol
+		(lib_id "power:+24V")
+		(at 27.94 135.89 180)
+		(unit 1)
+		(exclude_from_sim no)
+		(in_bom yes)
+		(on_board yes)
+		(dnp no)
+		(fields_autoplaced yes)
+		(property "Reference" "#PWR088"
+			(at 27.94 132.08 0)
+			(effects
+				(font
+					(size 1.27 1.27)
+				)
+				(hide yes)
+			)
+		)
+		(property "Value" "+24V"
+			(at 27.94 140.97 0)
+			(effects
+				(font
+					(size 1.27 1.27)
+				)
+			)
+		)
+		(property "Footprint" ""
+			(at 27.94 135.89 0)
+			(effects
+				(font
+					(size 1.27 1.27)
+				)
+				(hide yes)
+			)
+		)
+		(property "Datasheet" ""
+			(at 27.94 135.89 0)
+			(effects
+				(font
+					(size 1.27 1.27)
+				)
+				(hide yes)
+			)
+		)
+		(property "Description" "Power symbol creates a global label with name \"+24V\""
+			(at 27.94 135.89 0)
+			(effects
+				(font
+					(size 1.27 1.27)
+				)
+				(hide yes)
+			)
+		)
+		(pin "1"
+		)
+		(instances
+			(project "upper_lc_board_v2"
+				(path "/8de962ac-ee95-4233-a205-efbcd04063bc/94566a7d-86bb-4a04-89fe-f21a893d6a23"
+					(reference "#PWR088")
+					(unit 1)
+				)
+			)
+		)
+	)
+	(symbol
 		(lib_id "Device:FerriteBead")
 		(at 52.07 137.16 90)
@@
 			)
 		)
-		(property "Value" "24V-TP"
+		(property "Value" "24V-TP-P"
 			(at 72.898 135.636 0)
 			(effects
@@
 			)
 		)
-		(property "Footprint" "TestPoint:TestPoint_Pad_D1.0mm"
+		(property "Footprint" "TestPoint:TestPoint_Pad_1.5x1.5mm"
 			(at 76.2 137.16 0)
 			(effects

Commit message: review work
Parts:
- removed Q1: 2N7002, Package_TO_SOT_SMD:SOT-23, symbol Transistor_FET:2N7002
- removed R11, R13: 10k, Resistor_SMD:R_0603_1608Metric, symbol Device:R
- removed R12: 4.7k, Resistor_SMD:R_0603_1608Metric, symbol Device:R
- removed R14: 200, Resistor_SMD:R_0603_1608Metric, symbol Device:R
- removed U6: DMP4065S-7, Package_TO_SOT_SMD:SOT-23, symbol SI2301:SI2301CDS-T1-GE3
Other:
- note removed: "VSOL Switching"
