File: Schematics/upper_lc_board/modules/power_module/power_module.kicad_sch (KiCad schematic)
At the start: 29 parts, among them U3 LD1117S33TR_SOT223, U4 ID_LM66100DCKR, U5 ID_LM66100DCKR, U9 TVS3300DRV

Commit message: add requested changes for PR
Other:
- note added: "added a ferrite bead to form pi-filter to reduce propagation of noise throughout 24V branch during actuation"
- note added: "https://www.ti.com/lit/an/slva079/slva079.pdf?ts=1768142631143"
- note added: "switched to reccomended LDO based on lower Quiescent current (Iq)and greater PSSR a lower Iq increases efficiency."
- note removed: "reccomended LDO"
- moved on the sheet: C10, C13, C14, C9, D5, D?, F1, FB1, R9, R?, TP2, TP3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

Commit message: organizational work
Parts:
- added NT1: GND-TIE, NetTie:NetTie-2_SMD_Pad0.5mm, symbol Device:NetTie_2
- C10: JLCPCB (none) -> C14663
- C11, C12: JLCPCB (none) -> C15849
- C20, C?: value 100uF_16V -> 100uF
- C9: value 100uF_50V -> 100uF
- U3: value LD1117S33TR_SOT223 -> AMS1117; symbol Regulator_Linear:LD1117S33TR_SOT223 -> Regulator_Linear:AMS1117
Connections:
- net GND: now also NT1.2
- new net GNDA: NT1.1
Other:
- note added: "24V-LED: Vf=2.6, R=4.7k, I=4.5mA"
- note added: "3V3-LED: Vf=2.6, R=150, I=4.7mA"
- note added: "5V-LED: Vf=2.6, R=510, I=4.7mA"
- note added: "Analog GND Tie"
- note added: "PI-filter for filtering"
- note added: "Power LED Calculations"
- note removed: "Vf=2.6, R=4.7k, I=4.5mA"
- note removed: "Vf=2.6, R=510, I=4.7mA"
- note removed: "added a ferrite bead to form pi-filter to reduce propagation of noise throughout 24V branch during actuation"
- note removed: "https://www.ti.com/lit/an/slva079/slva079.pdf?ts=1768142631143"
- note removed: "switched to reccomended LDO based on lower Quiescent current (Iq)and greater PSSR a lower Iq increases efficiency."
- moved on the sheet: C10, C11, C12, C13, C14, C20, C9, C?, D5, D?, F1, FB1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

Commit message: more organizational work, add shared footprint, model, symbol dirs and clean up individuals
Parts:
- FB1: footprint BLM31KN121SN1L:BEADC3216X180N -> Resistor_SMD:R_0805_2012Metric
Other:
- title: ULC Board Power Circuitry -> PHEONIX | Power Circuitry
Changed lines of the file:
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@@
 	(paper "A4")
 	(title_block
-		(title "ULC Board Power Circuitry")
+		(title "PHEONIX | Power Circuitry")
 		(rev "A")
 		(company "Queen's Rocket Engineering Team")
@@
 			)
 		)
-		(property "Datasheet" "${KIPRJMOD}/../../Datasheets/ID-lm66100.pdf"
+		(property "Datasheet" "${KIPRJMOD}/../../Documentation/ideal_diode_lm66100_DS.pdf"
 			(at 177.8 74.93 0)
 			(effects
@@
 			)
 		)
-		(property "Footprint" "BLM31KN121SN1L:BEADC3216X180N"
+		(property "Footprint" "Resistor_SMD:R_0805_2012Metric"
 			(at 78.74 149.098 90)
 			(effects
@@
 			)
 		)
-		(property "Datasheet" "${KIPRJMOD}/../../Datasheets/FERRITEB-A700000010386127.pdf"
+		(property "Datasheet" ""
 			(at 78.74 147.32 0)
 			(effects
@@
 			)
 		)
-		(property "Datasheet" "http://www.advanced-monolithic.com/pdf/ds1117.pdf"
+		(property "Datasheet" "${KIPRJMOD}/../../Documentation/LDO_ds1117_DS.pdf"
 			(at 170.18 128.27 0)
 			(effects
@@
 			)
 		)
-		(property "Datasheet" "${KIPRJMOD}/../../Datasheets/ID-lm66100.pdf"
+		(property "Datasheet" "${KIPRJMOD}/../../Documentation/ideal_diode_lm66100_DS.pdf"
 			(at 177.8 52.07 0)
 			(effects
@@
 			)
 		)
-		(property "Datasheet" "${KIPRJMOD}/../../Datasheets/SURGE-PROT-tvs3300.pdf"
+		(property "Datasheet" "${KIPRJMOD}/../../Documentation/surgeprot_tvs3300_DS.pdf"
 			(at 60.96 154.94 0)
 			(effects

Commit message: increase width on power rails from USB and SWD, start tuning diff pairs
Parts:
- U3: Digikey (none) -> 5399-AMS1117-3.3SOT-223TR-ND
Changed lines of the file:
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@@
+			)
+		)
+		(property "Digikey" "5399-AMS1117-3.3SOT-223TR-ND"
+			(at 167.64 121.92 0)
+			(effects
+				(font
+					(size 1.27 1.27)
+				)
+				(hide yes)
 			)
 		)
