File: Schematics/upper_lc_board_v2/modules/actuation_module/actuation_module.kicad_sch (KiCad schematic)
At the start: 7 parts

Commit message: review work
Connections:
- net VSOL renamed +24V

Commit message: refactor with new conns
Parts:
- TP10, TP8: footprint TestPoint:TestPoint_Pad_D1.0mm -> TestPoint:TestPoint_Pad_1.5x1.5mm
Changed lines of the file:
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@@
 			)
 		)
-		(property "Footprint" "TestPoint:TestPoint_Pad_D1.0mm"
+		(property "Footprint" "TestPoint:TestPoint_Pad_1.5x1.5mm"
 			(at 165.1 78.74 0)
 			(effects
@@
 			)
 		)
-		(property "Footprint" "TestPoint:TestPoint_Pad_D1.0mm"
+		(property "Footprint" "TestPoint:TestPoint_Pad_1.5x1.5mm"
 			(at 162.56 124.46 0)
 			(effects
