File: Schematics/upper_lc_board_v2/esp32_breakout_module.kicad_sch (KiCad schematic)
At the start: 31 parts, among them J1 USB_C_Female_USB2_Small, Q4 2N7002, SW1 SW_ESP_BOOT_MODE, SW2 SW_ESP_RESET, U1 ESP32-S3-WROOM-1-N16, U2 ISO1044BDR

Commit message: layout updates after review, cleaned up schematic organization
Parts:
- removed R30: 470, Resistor_SMD:R_0603_1608Metric, symbol Device:R
Changed lines of the file:
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@@
 	)
 	(label "GPIO_42"
-		(at 80.01 151.13 90)
+		(at 95.25 153.67 90)
 		(fields_autoplaced yes)
 		(effects
@@
 					(unit 1)
 				)
-			)
-		)
-	)
-	(symbol
-		(lib_id "Device:R")
-		(at 80.01 154.94 0)
-		(unit 1)
-		(exclude_from_sim no)
-		(in_bom yes)
-		(on_board yes)
-		(dnp no)
-		(property "Reference" "R30"
-			(at 74.676 153.67 0)
-			(effects
-				(font
-					(size 1.27 1.27)
-				)
-				(justify left)
-			)
-		)
-		(property "Value" "470"
-			(at 74.676 156.21 0)
-			(effects
-				(font
-					(size 1.27 1.27)
-				)
-				(justify left)
-			)
-		)
-		(property "Footprint" "Resistor_SMD:R_0603_1608Metric"
-			(at 78.232 154.94 90)
-			(effects
-				(font
-					(size 1.27 1.27)
-				)
-				(hide yes)
-			)
-		)
-		(property "Datasheet" "~"
-			(at 80.01 154.94 0)
-			(effects
-				(font
-					(size 1.27 1.27)
-				)
-				(hide yes)
-			)
-		)
-		(property "Description" "Resistor"
-			(at 80.01 154.94 0)
-			(effects
-				(font
-					(size 1.27 1.27)
-				)
-				(hide yes)
-			)
-		)
-		(property "JLCPCB" "C23179"
-			(at 80.01 154.94 0)
-			(effects
-				(font
-					(size 1.27 1.27)
-				)
-				(hide yes)
-			)
-		)
-		(pin "1"
-		)
-		(pin "2"
-		)
-		(instances
-			(project "upper_lc_board_v2"
-				(path "/8de962ac-ee95-4233-a205-efbcd04063bc/fb03bfcd-cf55-42d7-9f53-690866bb15a9"
-					(reference "R30")
-					(unit 1)
-				)

Commit message: swap I2C lines, add digi numbers to conns, fix diode issue
Parts:
- R29: JLCPCB (none) -> C21190
Connections:
- net HALL_SCL: now also U1.10 (IO17); no longer U1.11 (IO18)
- net HALL_SDA: now also U1.11 (IO18); no longer U1.10 (IO17)
Changed lines of the file:
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@@
 	(global_label "HALL_SDA"
+		(shape input)
+		(at 194.31 97.79 0)
+		(fields_autoplaced yes)
+		(effects
+			(font
+				(size 1.27 1.27)
+			)
+			(justify left)
+		)
+		(property "Intersheetrefs" "${INTERSHEET_REFS}"
+			(at 206.3062 97.79 0)
+			(effects
+				(font
+					(size 1.27 1.27)
+				)
+				(justify left)
+				(hide yes)
+			)
+		)
+	)
+	(global_label "HALL_SCL"
 		(shape input)
 		(at 194.31 93.98 0)
@@
 		)
 		(property "Intersheetrefs" "${INTERSHEET_REFS}"
-			(at 206.3062 93.98 0)
+			(at 206.2457 93.98 0)
 			(effects
 				(font
@@
 		)
 	)
-	(global_label "HALL_SCL"
-		(shape input)
-		(at 194.31 97.79 0)
-		(fields_autoplaced yes)
-		(effects
-			(font
-				(size 1.27 1.27)
-			)
-			(justify left)
-		)
-		(property "Intersheetrefs" "${INTERSHEET_REFS}"
-			(at 206.2457 97.79 0)
-			(effects
-				(font
-					(size 1.27 1.27)
-				)
-				(justify left)
-				(hide yes)
-			)
-		)
-	)
 	(global_label "BUZZ_IN"
 		(shape input)
@@
 			(at 138.43 147.32 0)
 			(effects
+				(font
+					(size 1.27 1.27)
+				)
+				(hide yes)
+			)
+		)
+		(property "JLCPCB" "C21190"
+			(at 138.43 147.32 0)
+			(effects

Commit message: resolve DRC & tweak
Connections:
- net GPIO_42: now also D4.4 (DIN)
Changed lines of the file:
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@@
+	)
+	(no_connect
+		(at 80.01 158.75)
 	)
 	(no_connect
@@
 	(no_connect
 		(at 132.08 119.38)
-	)
-	(no_connect
-		(at 95.25 158.75)
 	)
 	(no_connect
@@
 	)
 	(label "GPIO_42"
-		(at 95.25 153.67 90)
-		(fields_autoplaced yes)
-		(effects
-			(font
-				(size 1.27 1.27)
-				(color 0 0 0 1)
-			)
-			(justify left bottom)
-		)
-	)
+		(at 95.25 158.75 270)
+		(fields_autoplaced yes)
+		(effects
+			(font
+				(size 1.27 1.27)
+				(color 0 0 0 1)
+			)
+			(justify right bottom)
+		)
+	)

Commit message: updated part numbers and fixed minor circuit issues
Parts:
- removed D15: 1N4148WS-7-F, Diode_SMD:D_SOD-323, symbol Diode:1N4148WS
- removed R27: 220, Resistor_SMD:R_0603_1608Metric, symbol Device:R
- removed R29: 1k, Resistor_SMD:R_0603_1608Metric, symbol Device:R
- added R10: 200, Resistor_SMD:R_0603_1608Metric, symbol Device:R
- BZ1: value Buzzer -> PS1240P02BT; footprint Buzzer_Beeper:Buzzer_TDK_PS1240P02BT_D12.2mm_H6.5mm -> footprints:Buzzer_12.6x9.5RM5.0; Digikey (none) -> 445-2525-1-ND; JLCPCB C76871 -> (none)
- C23, C27: JLCPCB C14663 -> (none); LCSC (none) -> C14663
- D1: value FAULT_LED -> FAULT_LED (RED); LCSC C2290 -> C2286
- D2: value CAN_LED -> CAN_LED (WHT)
- D3: value WIFI_LED -> WIFI_LED (WHT)
- J1: JLCPCB C5178541 -> (none); LCSC (none) -> C5178541
- Q4: JLCPCB C8545 -> (none); LCSC (none) -> C8545
- R2: value 150 -> 680; LCSC C22808 -> C23228
- R28: value 10K -> 10k; JLCPCB C25804 -> (none); LCSC (none) -> C25804
- R3, R4: value 150 -> 270; LCSC C22808 -> C22966
Connections:
- net +5V: now also C27.2; no longer C27.1
- net BUZZ_IN: now also R10.2
- net GND: now also C27.1; no longer C27.2
- net at Q4.1 (G), R28.2: now also R10.1
