File: Schematics/lower_lc_board/power_module.kicad_sch (KiCad schematic)
At the start: 34 parts, among them J1 Conn_01x06, U10 ID_LM66100DCKR, U2 AMS1117, U3 ID_LM66100DCKR, U4 ID_LM66100DCKR

Commit message: update backplane orientation
Parts:
- added C12: 10uF, Capacitor_SMD:C_0603_1608Metric, symbol Device:C
- U2: JLCPCB (none) -> C6186; LCSC (none) -> C6186
Connections:
- net 3V3_USB: now also C12.1
- net GND: now also C12.2

Commit message: PCB for review
Parts:
- removed C2: 0.1uF, Capacitor_SMD:C_0603_1608Metric, symbol Device:C
- removed FB1: FerriteBead, Resistor_SMD:R_0805_2012Metric, symbol Device:FerriteBead
- C51: LCSC (none) -> C1588
Connections:
- net +24V_BP: now also C3.1, F1.2
Other:
- note removed: "PI-filter for filtering"
- moved on the sheet: C3, D2, F1, R2, TP1

Commit message: WIP - i2c-2 refactor
Parts:
- C12, C7: JLCPCB C96446 -> (none)
- C44, C5, C6: JLCPCB C15849 -> (none)
- C50: JLCPCB C96446 -> (none); LCSC (none) -> C96446
- C51: JLCPCB C1588 -> (none)
- C52: JLCPCB C14663 -> (none); LCSC (none) -> C14663
- R1: JLCPCB C22962 -> (none)
- R2: JLCPCB C17936 -> (none); LCSC (none) -> C17936
- R3: JLCPCB C23186 -> (none)
- R4: JLCPCB C23138 -> (none)
- U10, U3, U4: JLCPCB C2869734 -> (none)
- U2: JLCPCB C6186 -> (none)
Changed lines of the file:
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@@
 			)
 		)
-		(property "JLCPCB" "C2869734"
-			(at 170.18 41.91 0)
-			(effects
-				(font
-					(size 1.27 1.27)
-				)
-				(hide yes)
-			)
-		)
 		(property "Sim.Device" ""
 			(at 170.18 41.91 0)
@@
 			)
 		)
-		(property "JLCPCB" "C96446"
-			(at 189.23 140.97 0)
-			(effects
-				(font
-					(size 1.27 1.27)
-				)
-				(hide yes)
-			)
-		)
 		(property "Sim.Device" ""
 			(at 189.23 140.97 0)
@@
 			)
 		)
-		(property "JLCPCB" "C23138"
-			(at 157.48 119.38 0)
-			(effects
-				(font
-					(size 1.27 1.27)
-				)
-				(hide yes)
-			)
-		)
 		(property "Sim.Device" ""
 			(at 157.48 119.38 0)
@@
 			)
 		)
-		(property "JLCPCB" "C22962"
-			(at 59.69 102.87 0)
-			(effects
-				(font
-					(size 1.27 1.27)
-				)
-				(hide yes)
-			)
-		)
 		(property "Sim.Device" ""
 			(at 59.69 102.87 0)
@@
 			)
 		)
-		(property "JLCPCB" "C96446"
+		(property "Sim.Device" ""
 			(at 204.47 69.85 0)
 			(effects
@@
 			)
 		)
-		(property "Sim.Device" ""
+		(property "Sim.Pins" ""
 			(at 204.47 69.85 0)
 			(effects
@@
 			)
 		)
-		(property "Sim.Pins" ""
+		(property "LCSC" "C96446"
 			(at 204.47 69.85 0)
 			(effects
@@
 			)
 		)
-		(property "JLCPCB" "C2869734"
-			(at 170.18 85.09 0)
-			(effects
-				(font
-					(size 1.27 1.27)
-				)
-				(hide yes)
-			)
-		)
 		(property "Sim.Device" ""
 			(at 170.18 85.09 0)
@@
 			)
 		)
-		(property "JLCPCB" "C23186"
-			(at 100.33 100.33 0)
-			(effects
-				(font
-					(size 1.27 1.27)
-				)
-				(hide yes)
-			)
-		)
 		(property "Sim.Device" ""
 			(at 100.33 100.33 0)
@@
 			)
 		)
-		(property "JLCPCB" "C15849"
-			(at 142.24 43.18 0)
-			(effects
-				(font
-					(size 1.27 1.27)
-				)
-				(hide yes)
-			)
-		)
 		(property "Sim.Device" ""
 			(at 142.24 43.18 0)
@@
 			)
 		)
-		(property "JLCPCB" "C96446"
-			(at 160.02 140.97 0)
-			(effects
-				(font
-					(size 1.27 1.27)
-				)
-				(hide yes)
-			)
-		)
 		(property "Sim.Device" ""
 			(at 160.02 140.97 0)
@@
 			)
 		)
-		(property "JLCPCB" "C2869734"
-			(at 170.18 64.77 0)
-			(effects
-				(font
-					(size 1.27 1.27)
-				)
-				(hide yes)
-			)
-		)
 		(property "Sim.Device" ""
 			(at 170.18 64.77 0)
@@
 			)
 		)
-		(property "JLCPCB" "C14663"
+		(property "Sim.Device" ""
 			(at 204.47 62.23 0)
 			(effects
@@
 			)
 		)
-		(property "Sim.Device" ""
+		(property "Sim.Pins" ""
 			(at 204.47 62.23 0)
 			(effects
@@
 			)
 		)
-		(property "Sim.Pins" ""
+		(property "LCSC" "C14663"
 			(at 204.47 62.23 0)
 			(effects
@@
 			)
 		)
-		(property "JLCPCB" "C1588"
-			(at 204.47 50.8 0)
-			(effects
-				(font
-					(size 1.27 1.27)
-				)
-				(hide yes)
-			)
-		)
 		(property "Sim.Device" ""
 			(at 204.47 50.8 0)
@@
 			)
 		)
-		(property "JLCPCB" "C15849"
-			(at 143.51 66.04 0)
-			(effects
-				(font
-					(size 1.27 1.27)
-				)
-				(hide yes)
-			)
-		)
 		(property "Sim.Device" ""
 			(at 143.51 66.04 0)
@@
 			)
 		)
-		(property "JLCPCB" "C17936"
+		(property "Sim.Device" ""
 			(at 80.01 138.43 0)
 			(effects
@@
 			)
 		)
-		(property "Sim.Device" ""
+		(property "Sim.Pins" ""
 			(at 80.01 138.43 0)
 			(effects
@@
 			)
 		)
-		(property "Sim.Pins" ""
+		(property "LCSC" "C17936"
 			(at 80.01 138.43 0)
 			(effects
@@
 			)
 		)
-		(property "JLCPCB" "C15849"
-			(at 143.51 86.36 0)
-			(effects
-				(font
-					(size 1.27 1.27)
-				)
-				(hide yes)
-			)
-		)
 		(property "Sim.Device" ""
 			(at 143.51 86.36 0)
@@
 			(at 168.91 137.16 0)
 			(effects
-				(font
-					(size 1.27 1.27)
-				)
-				(hide yes)
-			)
-		)
-		(property "JLCPCB" "C6186"
-			(at 168.91 137.16 0)
-			(effects

Commit message: start 2nd refactor
Parts:
- added R46: 120, Resistor_SMD:R_0603_1608Metric, symbol Device:R
- R2: value 4.7k -> 12k; footprint Resistor_SMD:R_1206_3216Metric_Pad1.30x1.75mm_HandSolder -> Resistor_SMD:R_0603_1608Metric; LCSC C17936 -> C22790
Connections:
- net CAN_N: now also R46.1
- net CAN_P: now also R46.2
Other:
- note added: "CANbus termination"
Changed lines of the file:
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@@
 		)
 	)
+	(text "CANbus termination"
+		(exclude_from_sim no)
+		(at 109.5622 76.5995 0)
+		(effects
+			(font
+				(size 1.27 1.27)
+				(thickness 0.254)
+				(bold yes)
+				(color 0 0 0 1)
+			)
+		)
+	)
 	(text "24V-LED: Vf=2.6, R=4.7k, I=4.5mA"
 		(exclude_from_sim no)
@@
 	(global_label "CAN_N"
 		(shape input)
+		(at 106.0062 65.1695 270)
+		(fields_autoplaced yes)
+		(effects
+			(font
+				(size 1.27 1.27)
+			)
+			(justify right)
+		)
+		(property "Intersheetrefs" "${INTERSHEET_REFS}"
+			(at 106.0062 74.1419 90)
+			(effects
+				(font
+					(size 1.27 1.27)
+				)
+				(justify right)
+				(hide yes)
+			)
+		)
+	)
+	(global_label "CAN_N"
+		(shape input)
 		(at 77.47 54.61 270)
 		(fields_autoplaced yes)
@@
 		)
 	)
+	(global_label "CAN_P"
+		(shape input)
+		(at 113.6262 65.1695 270)
+		(fields_autoplaced yes)
+		(effects
+			(font
+				(size 1.27 1.27)
+			)
+			(justify right)
+		)
+		(property "Intersheetrefs" "${INTERSHEET_REFS}"
+			(at 113.6262 74.0814 90)
+			(effects
+				(font
+					(size 1.27 1.27)
+				)
+				(justify right)
+				(hide yes)
+			)
+		)
+	)
 	(symbol
 		(lib_id "QRET_Buck_PSU:LM66100DCKR")
@@
 	)
 	(symbol
+		(lib_id "Device:R")
+		(at 109.8162 65.1695 90)
+		(unit 1)
+		(exclude_from_sim no)
+		(in_bom yes)
+		(on_board yes)
+		(dnp no)
+		(fields_autoplaced yes)
+		(property "Reference" "R46"
+			(at 109.8162 58.8195 90)
+			(effects
+				(font
+					(size 1.27 1.27)
+				)
+			)
+		)
+		(property "Value" "120"
+			(at 109.8162 61.3595 90)
+			(effects
+				(font
+					(size 1.27 1.27)
+				)
+			)
+		)
+		(property "Footprint" "Resistor_SMD:R_0603_1608Metric"
+			(at 109.8162 66.9475 90)
+			(effects
+				(font
+					(size 1.27 1.27)
+				)
+				(hide yes)
+			)
+		)
+		(property "Datasheet" "~"
+			(at 109.8162 65.1695 0)
+			(effects
+				(font
+					(size 1.27 1.27)
+				)
+				(hide yes)
+			)
+		)
+		(property "Description" "CAN Termination Resistor"
+			(at 109.8162 65.1695 0)
+			(effects
+				(font
+					(size 1.27 1.27)
+				)
+				(hide yes)
+			)
+		)
+		(property "LCSC" "C22787"
+			(at 109.8162 65.1695 0)
+			(effects
+				(font
+					(size 1.27 1.27)
+				)
+				(hide yes)
+			)
+		)
+		(pin "2"
+		)
+		(pin "1"
+		)
+		(instances
+			(project "lower_lc_board"
+				(path "/d63798c4-e363-437e-9012-e4aff32e6642/ea1dc739-d1f4-46a0-a090-2a1bf39da427"
+					(reference "R46")
+					(unit 1)
+				)
+			)
+		)
+	)
+	(symbol
 		(lib_id "Device:C")
 		(at 143.51 66.04 0)
@@
 			)
 		)
-		(property "Value" "4.7k"
+		(property "Value" "12k"
 			(at 80.01 138.43 90)
 			(effects
@@
 			)
 		)
-		(property "Footprint" "Resistor_SMD:R_1206_3216Metric_Pad1.30x1.75mm_HandSolder"
+		(property "Footprint" "Resistor_SMD:R_0603_1608Metric"
 			(at 81.788 138.43 90)
 			(effects
@@
 			)
 		)
-		(property "LCSC" "C17936"
+		(property "LCSC" "C22790"
 			(at 80.01 138.43 0)
 			(effects

Commit message: updates and added to cart
Parts:
- removed R4: 330, Resistor_SMD:R_0603_1608Metric, symbol Device:R
- removed R46: 120, Resistor_SMD:R_0603_1608Metric, symbol Device:R
- added R16: 6.2k, Resistor_SMD:R_0603_1608Metric, symbol Device:R
- D1, D2, D3, D4: Digikey 150080VS75000 -> (none)
- J1: footprint CONN_SD-4:CONN_SD-43045-001_06_MOL -> CONN_SD-4:CONN_SD-105314-100_06_MOL
- R1: value 220 -> 3.3k; LCSC C22808 -> C22978
- R3: value 510 -> 6.2k; LCSC C23193 -> C4260
- U2: value AMS1117 -> AMS1117-3.3; Digikey 5399-AMS1117-3.3SOT-223TR-ND -> (none)
Connections:
- net +3V3: now also R1.1; no longer R1.2
- net 5V_USB: now also R16.1
- net at D4.2 (A): now also R16.2
- net at D1.2 (A): now also R1.2; no longer R1.1
Other:
- note removed: "CANbus termination"

Commit message: add board-specifc READMEs (TODO), cleanup schematic titles
Other:
- title: HYDRA | Power Circuitry -> Power Management Circuitry
Changed lines of the file:
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@@
 	(paper "A4")
 	(title_block
-		(title "HYDRA | Power Circuitry")
+		(title "Power Management Circuitry")
 		(rev "2")
 		(company "Queen's Rocket Engineering Team")
-		(comment 1 "Jeevan Sanchez")
+		(comment 1 "Contributors: Jeevan Sanchez, Tristan Alderson")
+		(comment 2 "HYDRA - Lower Control Board")
 	)
 	(junction
