File: Schematics/lower_lc_board/actuation_module.kicad_sch (KiCad schematic)
At the start: 13 parts, among them Q5 2N7002, U12 DMP4065S-7

Commit message: WIP - i2c-2 refactor
Parts:
- D11, D12: JLCPCB C2290 -> (none)
- Q5: JLCPCB C8545 -> (none)
- R30, R31: value 4.7k -> 12k; JLCPCB C17936 -> (none); LCSC (none) -> C17912
- R50, R52: JLCPCB C25804 -> (none); LCSC (none) -> C25804
- R51: value 4.7k -> 6.2K; JLCPCB C23162 -> (none); LCSC (none) -> C4260
- R53: JLCPCB C8218 -> (none); LCSC (none) -> C8218
- U12: JLCPCB C182476 -> (none)
Changed lines of the file:
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@@
-			)
-		)
-		(property "JLCPCB" ""
-			(at 229.87 55.88 0)
-			(effects
-				(font
-					(size 1.27 1.27)
-				)
-				(hide yes)
 			)
 		)
@@
 			)
 		)
-		(property "Value" "4.7k"
+		(property "Value" "12k"
 			(at 102.87 76.2 90)
 			(effects
@@
 			)
 		)
-		(property "JLCPCB" "C17936"
-			(at 102.87 76.2 0)
-			(effects
-				(font
-					(size 1.27 1.27)
-				)
-				(hide yes)
-			)
-		)
 		(property "Sim.Device" ""
 			(at 102.87 76.2 0)
@@
 			)
 		)
+		(property "LCSC" "C17912"
+			(at 102.87 76.2 0)
+			(effects
+				(font
+					(size 1.27 1.27)
+				)
+				(hide yes)
+			)
+		)
 		(pin "2"
 		)
@@
 			)
 		)
-		(property "JLCPCB" "C25804"
-			(at 71.12 119.38 0)
-			(effects
-				(font
-					(size 1.27 1.27)
-				)
-				(hide yes)
-			)
-		)
 		(property "Sim.Device" ""
 			(at 71.12 119.38 0)
@@
 			)
 		)
+		(property "LCSC" "C25804"
+			(at 71.12 119.38 0)
+			(effects
+				(font
+					(size 1.27 1.27)
+				)
+				(hide yes)
+			)
+		)
 		(pin "1"
 		)
@@
 			)
 		)
-		(property "JLCPCB" "C25804"
-			(at 87.63 114.3 0)
-			(effects
-				(font
-					(size 1.27 1.27)
-				)
-				(hide yes)
-			)
-		)
 		(property "Sim.Device" ""
 			(at 87.63 114.3 0)
@@
 			)
 		)
+		(property "LCSC" "C25804"
+			(at 87.63 114.3 0)
+			(effects
+				(font
+					(size 1.27 1.27)
+				)
+				(hide yes)
+			)
+		)
 		(pin "1"
 		)
@@
 			)
 		)
-		(property "JLCPCB" "C8218"
-			(at 93.98 110.49 0)
-			(effects
-				(font
-					(size 1.27 1.27)
-				)
-				(hide yes)
-			)
-		)
 		(property "Sim.Device" ""
 			(at 93.98 110.49 0)
@@
 			)
 		)
+		(property "LCSC" "C8218"
+			(at 93.98 110.49 0)
+			(effects
+				(font
+					(size 1.27 1.27)
+				)
+				(hide yes)
+			)
+		)
 		(pin "1"
 		)
@@
 		)
 		(property "Sim.Pins" ""
-			(at 82.55 125.73 0)
-			(effects
-				(font
-					(size 1.27 1.27)
-				)
-				(hide yes)
-			)
-		)
-		(property "JLCPCB" "C182476"
 			(at 82.55 125.73 0)
 			(effects
@@
 			)
 		)
-		(property "Value" "4.7k"
+		(property "Value" "6.2K"
 			(at 83.058 119.38 90)
 			(effects
@@
 			)
 		)
-		(property "JLCPCB" "C23162"
-			(at 81.28 119.38 0)
-			(effects
-				(font
-					(size 1.27 1.27)
-				)
-				(hide yes)
-			)
-		)
 		(property "Sim.Device" ""
 			(at 81.28 119.38 0)
@@
 			)
 		)
+		(property "LCSC" "C4260"
+			(at 81.28 119.38 0)
+			(effects
+				(font
+					(size 1.27 1.27)
+				)
+				(hide yes)
+			)
+		)
 		(pin "1"
 		)
@@
 			)
 		)
-		(property "Value" "4.7k"
+		(property "Value" "12k"
 			(at 102.87 60.96 90)
 			(effects
@@
 			)
 		)
-		(property "JLCPCB" "C17936"
-			(at 102.87 60.96 0)
-			(effects
-				(font
-					(size 1.27 1.27)
-				)
-				(hide yes)
-			)
-		)
 		(property "Sim.Device" ""
 			(at 102.87 60.96 0)
@@
 		)
 		(property "Sim.Pins" ""
+			(at 102.87 60.96 0)
+			(effects
+				(font
+					(size 1.27 1.27)
+				)
+				(hide yes)
+			)
+		)
+		(property "LCSC" "C17912"
 			(at 102.87 60.96 0)
 			(effects
@@
 			)
 		)
-		(property "JLCPCB" "C8545"
-			(at 76.2 105.41 0)
-			(effects
-				(font
-					(size 1.27 1.27)
-				)
-				(hide yes)
-			)
-		)
 		(property "Sim.Device" ""
 			(at 76.2 105.41 0)
@@
 			)
 		)
-		(property "JLCPCB" "C2290"
-			(at 95.25 76.2 0)
-			(effects
-				(font
-					(size 1.27 1.27)
-				)
-				(hide yes)
-			)
-		)
 		(property "Sim.Device" ""
 			(at 95.25 76.2 0)
@@
 			(at 95.25 60.96 0)
 			(effects
-				(font
-					(size 1.27 1.27)
-				)
-				(hide yes)
-			)
-		)
-		(property "JLCPCB" "C2290"
-			(at 95.25 60.96 0)
-			(effects

Commit message: start 2nd refactor
Parts:
- R30, R31: footprint Resistor_SMD:R_1206_3216Metric_Pad1.30x1.75mm_HandSolder -> Resistor_SMD:R_0603_1608Metric; LCSC C17912 -> C22790
Other:
- note removed: "added to avoid constant power drain"
Changed lines of the file:
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@@
-		)
-	)
-	(text "added to avoid constant power drain"
-		(exclude_from_sim no)
-		(at 103.886 94.234 0)
-		(effects
-			(font
-				(size 0.889 0.889)
-				(color 0 0 0 1)
-			)
-			(justify left)
 		)
 	)
@@
 			)
 		)
-		(property "Footprint" "Resistor_SMD:R_1206_3216Metric_Pad1.30x1.75mm_HandSolder"
+		(property "Footprint" "Resistor_SMD:R_0603_1608Metric"
 			(at 102.87 77.978 90)
 			(effects
@@
 			)
 		)
-		(property "LCSC" "C17912"
+		(property "LCSC" "C22790"
 			(at 102.87 76.2 0)
 			(effects
@@
 		)
 		(property "Value" "6.2K"
-			(at 83.058 119.38 90)
+			(at 83.566 119.38 90)
 			(effects
 				(font
@@
 			)
 		)
-		(property "Footprint" "Resistor_SMD:R_1206_3216Metric_Pad1.30x1.75mm_HandSolder"
+		(property "Footprint" "Resistor_SMD:R_0603_1608Metric"
 			(at 102.87 62.738 90)
 			(effects
@@
 			)
 		)
-		(property "LCSC" "C17912"
+		(property "LCSC" "C22790"
 			(at 102.87 60.96 0)
 			(effects

Commit message: change TP footprint for consistency across boards
Parts:
- TP11, TP12: footprint TestPoint:TestPoint_Pad_D1.0mm -> TestPoint:TestPoint_Pad_1.0x1.0mm
Changed lines of the file:
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@@
 			)
 		)
-		(property "Footprint" "TestPoint:TestPoint_Pad_D1.0mm"
+		(property "Footprint" "TestPoint:TestPoint_Pad_1.0x1.0mm"
 			(at 160.02 76.2 0)
 			(effects
@@
 			)
 		)
-		(property "Footprint" "TestPoint:TestPoint_Pad_D1.0mm"
+		(property "Footprint" "TestPoint:TestPoint_Pad_1.0x1.0mm"
 			(at 157.48 121.92 0)
 			(effects

Commit message: updates and added to cart
Parts:
- removed TP11: VALVE1_OUT_TP, TestPoint:TestPoint_Pad_1.0x1.0mm, symbol Connector:TestPoint
- removed TP12: VALVE2_OUT_TP, TestPoint:TestPoint_Pad_1.0x1.0mm, symbol Connector:TestPoint
- added R47: 100k, Resistor_SMD:R_0603_1608Metric, symbol Device:R
- added R54: 10k, Resistor_SMD:R_0603_1608Metric, symbol Device:R
- added TP7: VSOL.S, TestPoint:TestPoint_Pad_1.5x1.5mm, symbol Connector:TestPoint
- R51: value 6.2K -> 6.2k
Connections:
- net GND: now also R54.1
- net VSOL: now also R47.1
- new net VSOL_SENSE: R47.2, R54.2, TP7.1
Other:
- sheet Valve Control 1 ports: added none; removed TP
- sheet Valve Control 2 ports: added none; removed TP
- note removed: "Bulk Decoupling"
- title: HYDRA | Actuation Circuitry -> QRET 25-26 SRAD Hyrbid Lower Control Module
- moved on the sheet: C46

Commit message: add board-specifc READMEs (TODO), cleanup schematic titles
Other:
- title: QRET 25-26 SRAD Hyrbid Lower Control Module -> Solenoid Driver Circuitry
Changed lines of the file:
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@@
 	(paper "A4")
 	(title_block
-		(title "QRET 25-26 SRAD Hyrbid Lower Control Module")
+		(title "Solenoid Driver Circuitry")
 		(rev "V1.0")
 		(company "Queen's Rocket Engineering Team")
 		(comment 1 "Contributors: Jeevan Sanchez, Tristan Alderson")
+		(comment 2 "HYDRA - Lower Control Board")
 	)
 	(junction

Commit message: add ed pinouts
Connections:
- net VSOL-SW renamed VSOL_EN
Changed lines of the file:
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@@
 		)
 	)
-	(global_label "VALVE2_CTRL"
+	(global_label "SOL2_EN"
 		(shape input)
 		(at 157.48 120.65 180)
@@
 		)
 		(property "Intersheetrefs" "${INTERSHEET_REFS}"
-			(at 142.3391 120.65 0)
+			(at 146.2701 120.65 0)
 			(effects
 				(font
@@
 		)
 	)
-	(global_label "VALVE1_CTRL"
+	(global_label "SOL1_EN"
 		(shape input)
 		(at 160.02 74.93 180)
@@
 		)
 		(property "Intersheetrefs" "${INTERSHEET_REFS}"
-			(at 144.8791 74.93 0)
+			(at 148.8101 74.93 0)
 			(effects
 				(font
@@
 		)
 	)
-	(global_label "VSOL-SW"
+	(global_label "VSOL_EN"
 		(shape input)
 		(at 97.79 110.49 0)
@@
 		)
 		(property "Intersheetrefs" "${INTERSHEET_REFS}"
-			(at 109.6652 110.49 0)
+			(at 108.879 110.49 0)
 			(effects
 				(font
